Commit message: - did a comparison with udemy plugin code

File: src/my_robot_description/urdf/ma_robot.ros2_control.xacro (robot description, xacro)
@@ -1,5 +1,5 @@
 <?xml version="1.0"?>
 <robot xmlns:xacro="http://www.ros.org/wiki/xacro">
-    <ros2_control name="my_arm_gripper" type="system">
+    <ros2_control name="ma_robot_arm" type="system">
         <hardware>
             <!--plugin>mock_components/GenericSystem</plugin-->
@@ -9,10 +9,4 @@
             <param name="joint3_servo_channel">13</param>
         </hardware>
-        <joint name="gripper_left_finger_joint">
-            <command_interface name="position"/>
-            <state_interface name="position">
-                <param name="initial_value">0.0</param>
-            </state_interface>
-        </joint>
         <joint name="joint1">
             <command_interface name="position"/>
@@ -52,3 +46,14 @@
         </joint>
     </ros2_control>
+    <ros2_control name="ma_robot_gripper" type="system">
+        <hardware>
+            <plugin>mock_components/GenericSystem</plugin>
+        </hardware>
+        <joint name="gripper_left_finger_joint">
+            <command_interface name="position"/>
+            <state_interface name="position">
+                <param name="initial_value">0.0</param>
+            </state_interface>
+        </joint>
+    </ros2_control>
 </robot>
