Commit message: - initial ros_control setup that connects moveit2 to fireware

File: src/my_robot_description/urdf/my_robot.urdf.xacro (robot description, xacro)
@@ -1,5 +1,6 @@
 <?xml version="1.0"?>
 <robot name="my_robot" xmlns:xacro="http://www.ros.org/wiki/xacro">
-    <xacro:include filename="common_properties.xacro" />
-    <xacro:include filename="my_robot_leg.xacro" />
+    <xacro:include filename="common_properties.xacro"/>
+    <xacro:include filename="my_robot_leg.xacro"/>
+    <xacro:include filename="my_robot.ros2_control.xacro"/>
 </robot>

File: src/my_robot_description/urdf/my_robot_leg.xacro (robot description, xacro)
@@ -287,5 +287,5 @@
         <origin xyz="${-servo_z/2-0.002-0.0025} ${-0.01-0.0025/2} 0" rpy="0 0 0"/>
         <axis xyz="1 0 0"/>
-        <mimic joint="servo3_calfFeet" multiplier="1.0" offset="0.0"/>
+        <!--mimic joint="servo3_calfFeet" multiplier="1.0" offset="0.0"/-->
         <limit effort="1000.0" velocity="1.0" lower="${5*urdf_pi/8}" upper="${11*urdf_pi/8}"/>
         <dynamics friction="0.05" damping="0.1"/>
