Commit message: - updated my_robot_commander.cpp; next to test the leg control with actual dynamixels - updated my_robot.gazebo.xacro; next to test the leg control with gazebo

File: src/my_robot_description/urdf/my_robot.gazebo.xacro (robot description, xacro)
@@ -1,14 +1,32 @@
 <?xml version="1.0"?>
-<robot name="ma_robot" xmlns:xacro="http://www.ros.org/wiki/xacro">
+<robot name="my_robot" xmlns:xacro="http://www.ros.org/wiki/xacro">
     <xacro:include filename="common_properties.xacro" />
     <xacro:include filename="my_robot_leg.xacro" />
+    <ros2_control name="GazeboInterface" type="system">
+        <hardware>
+            <plugin>gz_ros2_control/GazeboSimSystem</plugin>
+        </hardware>
+        <joint name="servo1_servo1_padding">
+                <command_interface name="position"/>
+                <state_interface name="position">
+                  <param name="initial_value">3.14</param>
+                </state_interface>
+            </joint>
+            <joint name="servo2_servo2_padding">
+                <command_interface name="position"/>
+                <state_interface name="position">
+                  <param name="initial_value">3.14</param>
+                </state_interface>
+            </joint>
+            <joint name="servo3_calfFeet">
+                <command_interface name="position"/>
+                <state_interface name="position">
+                  <param name="initial_value">3.14</param>
+                </state_interface>
+            </joint>
+    </ros2_control>
     <gazebo>
-        <plugin
-            filename="gz-sim-joint-state-publisher-system"
-            name="gz::sim::systems::JointStatePublisher">
-            <topic>joint_states</topic>
-            <topic_name>servo1_servo1_padding</topic_name>
-            <topic_name>servo2_servo2_padding</topic_name>
-            <topic_name>servo3_calfJoint</topic_name>
+        <plugin filename="gz_ros2_control-system" name="gz_ros2_control::GazeboSimROS2ControlPlugin">
+            <parameters>$(find my_robot_bringup)/config/my_robot_controllers.yaml</parameters>
         </plugin>
     </gazebo>
