Commit message: - updating all to run: ros2 launch my_robot_bringup my_robot.launch.py

File: src/my_robot_description/urdf/my_robot.ros2_control.xacro (robot description, xacro)
@@ -2,5 +2,4 @@
 <robot xmlns:xacro="http://www.ros.org/wiki/xacro">
     <xacro:macro name="my_robot_ros2_control" params="name initial_positions_file">
-        <xacro:property name="initial_positions" value="${xacro.load_yaml(initial_positions_file)['initial_positions']}"/>
         <ros2_control name="${name}" type="system">
             <hardware>
@@ -11,5 +10,5 @@
                 <command_interface name="position"/>
                 <state_interface name="position">
-                  <param name="initial_value">${initial_positions['servo1_servo1_padding']}</param>
+                  <param name="initial_value">3.14</param>
                 </state_interface>
             </joint>
@@ -17,5 +16,5 @@
                 <command_interface name="position"/>
                 <state_interface name="position">
-                  <param name="initial_value">${initial_positions['servo2_servo2_padding']}</param>
+                  <param name="initial_value">3.14</param>
                 </state_interface>
             </joint>
@@ -23,5 +22,5 @@
                 <command_interface name="position"/>
                 <state_interface name="position">
-                  <param name="initial_value">${initial_positions['servo3_calfFeet']}</param>
+                  <param name="initial_value">3.14</param>
                 </state_interface>
             </joint>

File: src/my_robot_description/urdf/my_robot.urdf.xacro (robot description, xacro)
@@ -1,6 +1,6 @@
 <?xml version="1.0"?>
 <robot name="my_robot" xmlns:xacro="http://www.ros.org/wiki/xacro">
-    <xacro:include filename="common_properties.xacro"/>
-    <xacro:include filename="my_robot_leg.xacro"/>
-    <xacro:include filename="my_robot.ros2_control.xacro"/>
+    <xacro:include filename="common_properties.xacro" />
+    <xacro:include filename="my_robot_leg.xacro" />
+    <xacro:include filename="my_robot.ros2_control.xacro" />
 </robot>

File: src/my_robot_description/urdf/my_robot_leg.xacro (robot description, xacro)
@@ -287,5 +287,5 @@
         <origin xyz="${-servo_z/2-0.002-0.0025} ${-0.01-0.0025/2} 0" rpy="0 0 0"/>
         <axis xyz="1 0 0"/>
-        <!--mimic joint="servo3_calfFeet" multiplier="1.0" offset="0.0"/-->
+        <mimic joint="servo3_calfFeet" multiplier="1.0" offset="0.0"/>
         <limit effort="1000.0" velocity="1.0" lower="${5*urdf_pi/8}" upper="${11*urdf_pi/8}"/>
         <dynamics friction="0.05" damping="0.1"/>

Commit message: - debugging my_robot_commander.cpp and hardware_interface_my_robot_dynamixel_u2d2_xl430.cpp; need safer way to run dynamixels

File: src/my_robot_description/urdf/my_robot.ros2_control.xacro (robot description, xacro)
@@ -1,32 +1,30 @@
 <?xml version="1.0"?>
 <robot xmlns:xacro="http://www.ros.org/wiki/xacro">
-    <xacro:macro name="my_robot_ros2_control" params="name initial_positions_file">
-        <ros2_control name="${name}" type="system">
-            <hardware>
-                <!--plugin>mock_components/GenericSystem</plugin-->
-                <plugin>my_robot_namespace/HardwareInterfaceU2D2_my_robot</plugin>
-                <param name="servo1_channel">11</param>
-                <param name="servo2_channel">12</param>
-                <param name="servo3_channel">13</param>
-            </hardware>
-            <joint name="servo1_servo1_padding">
-                <command_interface name="position"/>
-                <state_interface name="position">
-                  <param name="initial_value">3.14</param>
-                </state_interface>
-            </joint>
-            <joint name="servo2_servo2_padding">
-                <command_interface name="position"/>
-                <state_interface name="position">
-                  <param name="initial_value">3.14</param>
-                </state_interface>
-            </joint>
-            <joint name="servo3_calfFeet">
-                <command_interface name="position"/>
-                <state_interface name="position">
-                  <param name="initial_value">3.14</param>
-                </state_interface>
-            </joint>
-        </ros2_control>
-    </xacro:macro>
+    <ros2_control name="my_robot_controller" type="system">
+        <hardware>
+            <!--plugin>mock_components/GenericSystem</plugin-->
+            <plugin>my_robot_namespace/HardwareInterfaceU2D2_my_robot</plugin>
+            <param name="servo1_channel">11</param>
+            <param name="servo2_channel">12</param>
+            <param name="servo3_channel">13</param>
+        </hardware>
+        <joint name="servo1_servo1_padding">
+            <command_interface name="position"/>
+            <state_interface name="position">
+              <param name="initial_value">3.14</param>
+            </state_interface>
+        </joint>
+        <joint name="servo2_servo2_padding">
+            <command_interface name="position"/>
+            <state_interface name="position">
+              <param name="initial_value">3.14</param>
+            </state_interface>
+        </joint>
+        <joint name="servo3_calfFeet">
+            <command_interface name="position"/>
+            <state_interface name="position">
+              <param name="initial_value">3.14</param>
+            </state_interface>
+        </joint>
+    </ros2_control>
 </robot>

Commit message: - update the firmware such it also read out the velocity and effort (current) from dynamixel

File: src/my_robot_description/urdf/my_robot.ros2_control.xacro (robot description, xacro)
@@ -14,4 +14,10 @@
               <param name="initial_value">3.14</param>
             </state_interface>
+            <state_interface name="velocity">
+              <param name="initial_value">0.0</param>
+            </state_interface>
+            <state_interface name="effort">
+              <param name="initial_value">0.0</param>
+            </state_interface>
         </joint>
         <joint name="servo2_servo2_padding">
@@ -19,4 +25,10 @@
             <state_interface name="position">
               <param name="initial_value">3.14</param>
+            </state_interface>
+            <state_interface name="velocity">
+              <param name="initial_value">0.0</param>
+            </state_interface>
+            <state_interface name="effort">
+              <param name="initial_value">0.0</param>
             </state_interface>
         </joint>
@@ -26,4 +38,10 @@
               <param name="initial_value">3.14</param>
             </state_interface>
+            <state_interface name="velocity">
+              <param name="initial_value">0.0</param>
+            </state_interface>
+            <state_interface name="effort">
+              <param name="initial_value">0.0</param>
+            </state_interface>
         </joint>
     </ros2_control>

File: src/my_robot_description/urdf/my_robot_leg.xacro (robot description, xacro)
@@ -1,5 +1,5 @@
 <?xml version="1.0"?>
 <!-- ================================================================================================================================== -->
-<robot xmlns:xacro="http://www.ros.org/wiki/xacro" name="my_robot_leg">
+<robot xmlns:xacro="http://www.ros.org/wiki/xacro" name="my_robot">
     <xacro:property name="servo_x" value="0.0285"/>
     <xacro:property name="servo_y" value="0.0465"/>
@@ -289,5 +289,5 @@
                            o_xyz="-0.0005 0 0.0145" o_rpy="${urdf_pi/2} 0 ${-urdf_pi/2}"/>
     </link>
-    <joint name="servo3_calfJoint" type="revolute">
+    <!--joint name="servo3_calfJoint" type="revolute">
         <parent link="servo3"/>
         <child  link="calfJoint"/>
@@ -297,4 +297,9 @@
         <limit effort="1000.0" velocity="1.0" lower="${5*urdf_pi/8}" upper="${11*urdf_pi/8}"/>
         <dynamics friction="0.05" damping="0.1"/>
+    </joint-->
+    <joint name="servo3_calfJoint" type="fixed">
+        <parent link="servo3"/>
+        <child  link="calfJoint"/>
+        <origin xyz="${-servo_z/2-0.002-0.0025} ${-0.01-0.0025/2} 0" rpy="0 0 0"/>
     </joint>
     <link name="calfSphere">

File: src/my_robot_description/urdf/my_robot_leg_test.xacro (robot description, xacro)
@@ -1,5 +1,5 @@
 <?xml version="1.0"?>
 <!-- ================================================================================================================================== -->
-<robot xmlns:xacro="http://www.ros.org/wiki/xacro" name="my_robot_leg">
+<robot xmlns:xacro="http://www.ros.org/wiki/xacro" name="my_robot">
     <xacro:property name="effort"   value="30.0"/>
     <xacro:property name="velocity" value="10.0"/>
