Commit message: - trying to launch initial urdf with vis

File: src/my_robot_description/urdf/my_robot_leg.xacro (robot description, xacro)
@@ -2,5 +2,4 @@
 <!-- ================================================================================================================================== -->
 <robot xmlns:xacro="http://www.ros.org/wiki/xacro" name="my_robot_leg">
-    <xacro:include filename="$(find my_robot_description)/urdf/common_properties.xacro"/>
     <xacro:property name="effort"   value="30.0"/>
     <xacro:property name="velocity" value="10.0"/>
@@ -9,6 +8,4 @@
     <xacro:property name="servo_z" value="0.034"/>
 <!-- ================================================================================================================================== -->
-    <link name="world"/>
-    <!-- ============================ -->
     <link name="base_link">
         <visual>
@@ -16,12 +13,12 @@
                 <mesh filename="package://my_robot_description/mesh/CADv0/_mod_basePlate-Body.stl" scale="1.0 1.0 1.0"/>
             </geometry>
-            <origin rpy="0 0 0" xyz="0 0 0"/>
+            <origin xyz="0 0 0" rpy="0 0 0"/>
             <material name="white"/>
         </visual>
         <collision>
             <geometry>
-                <mesh filename="package://my_robot_description/mesh/CADv0/_mod_basePlate-Body.stl" scale="1.0 1.0 1.0"/>
+                <box size="0.1 0.1 0.004"/>
             </geometry>
-            <origin rpy="0 0 0" xyz="0 0 0"/>
+            <origin xyz="0 0 -0.002" rpy="0 0 0"/>
         </collision>
         <xacro:lazy_inertia m="1.0"/>
@@ -34,11 +31,11 @@
             </geometry>
             <material name="grey"/>
-            <origin rpy="0 0 0" xyz="0 0 0"/>
+            <origin xyz="0 0 0" rpy="0 0 0"/>
         </visual>
         <collision>
             <geometry>
-                <mesh filename="package://my_robot_description/mesh/CADv0/_mod_XL-430holderBasic.stl" scale="1.0 1.0 1.0"/>
+                <box size="0.037 0.032 0.014"/>
             </geometry>
-            <origin rpy="0 0 0" xyz="0 0 0"/>
+            <origin xyz="0 0 -0.007" rpy="0 0 0"/>
         </collision>
         <xacro:box_inertia m="0.01" x="0.037" y="0.032" z="0.014" o_xyz="0 0 -0.01" o_rpy="0 0 0"/>
@@ -47,7 +44,7 @@
         <parent link="base_link"/>
         <child  link="servo1_holder"/>
-        <origin xyz="0 0 0.004" rpy="0 0 0"/>
+        <origin xyz="0 0 0" rpy="0 0 0"/>
     </joint>
-    <link name="servo1">
+    <!--link name="servo1">
         <visual>
             <geometry>
@@ -61,5 +58,5 @@
                 <box size="${servo_x} ${servo_y} ${servo_z}"/>
             </geometry>
-            <origin rpy="0 0 0" xyz="0 0 0"/>
+            <origin xyz="0 0 0" rpy="0 0 0"/>
         </collision>
         <xacro:box_inertia m="0.0572" x="${servo_x}" y="${servo_y}" z="${servo_z}" o_xyz="0 0 0" o_rpy="0 0 0"/>
@@ -82,7 +79,7 @@
                 <cylinder radius="0.011" length="0.004"/>
             </geometry>
-            <origin rpy="0 0 0" xyz="0 0 0"/>
+            <origin xyz="0 0 0" rpy="0 0 0"/>
         </collision>
-        <xacro:cylinder_inertia m="0.001" x="0.011" l="0.004" o_xyz="0 0 0" o_rpy="0 0 0"/>
+        <xacro:cylinder_inertia m="0.001" r="0.011" l="0.004" o_xyz="0 0 0" o_rpy="0 0 0"/>
     </link>
     <joint name="servo1_servo1_padding" type="continuous">
@@ -92,5 +89,5 @@
         <axis xyz="0 1 0"/>
     </joint>
-    <!-- ============================ -->
+    < ============================ -->
 </robot>
 <!-- ================================================================================================================================== -->

Commit message: - experiencing not able to load mesh problem

File: src/my_robot_description/urdf/my_robot_leg.xacro (robot description, xacro)
@@ -11,5 +11,5 @@
         <visual>
             <geometry>
-                <mesh filename="package://my_robot_description/mesh/CADv0/_mod_basePlate-Body.stl" scale="1.0 1.0 1.0"/>
+                <mesh filename="/home/kali/Documents/ROS_init_practice/ros2_ws5_manipulator/src/my_robot_description/mesh/basement.STL"/>
             </geometry>
             <origin xyz="0 0 0" rpy="0 0 0"/>

Commit message: - resolving the mesh not loading problem

File: src/my_robot_description/urdf/my_robot_leg.xacro (robot description, xacro)
@@ -11,5 +11,5 @@
         <visual>
             <geometry>
-                <mesh filename="/home/kali/Documents/ROS_init_practice/ros2_ws5_manipulator/src/my_robot_description/mesh/basement.STL"/>
+                <mesh filename="package://my_robot_description/mesh/CADv0/_mod_basePlate-Body.stl" scale="1.0 1.0 1.0"/>
             </geometry>
             <origin xyz="0 0 0" rpy="0 0 0"/>
@@ -18,5 +18,5 @@
         <collision>
             <geometry>
-                <box size="0.1 0.1 0.004"/>
+                <mesh filename="package://my_robot_description/mesh/CADv0/_mod_basePlate-Body.stl" scale="1.0 1.0 1.0"/>
             </geometry>
             <origin xyz="0 0 -0.002" rpy="0 0 0"/>
@@ -28,5 +28,5 @@
         <visual>
             <geometry>
-                <mesh filename="package://my_robot_description/mesh/CADv0/_mod_XL-430holderBasic.stl" scale="1.0 1.0 1.0"/>
+                <mesh filename="package://my_robot_description/mesh/CADv0/_mod_XL-430holderBasic-Body.stl" scale="1.0 1.0 1.0"/>
             </geometry>
             <material name="grey"/>
@@ -35,5 +35,5 @@
         <collision>
             <geometry>
-                <box size="0.037 0.032 0.014"/>
+                <mesh filename="package://my_robot_description/mesh/CADv0/_mod_XL-430holderBasic-Body.stl" scale="1.0 1.0 1.0"/>
             </geometry>
             <origin xyz="0 0 -0.007" rpy="0 0 0"/>

Commit message: - urdf up to the first servo

File: src/my_robot_description/urdf/my_robot_leg.xacro (robot description, xacro)
@@ -2,6 +2,4 @@
 <!-- ================================================================================================================================== -->
 <robot xmlns:xacro="http://www.ros.org/wiki/xacro" name="my_robot_leg">
-    <xacro:property name="effort"   value="30.0"/>
-    <xacro:property name="velocity" value="10.0"/>
     <xacro:property name="servo_x" value="0.0285"/>
     <xacro:property name="servo_y" value="0.0465"/>
@@ -11,14 +9,14 @@
         <visual>
             <geometry>
-                <mesh filename="package://my_robot_description/mesh/CADv0/_mod_basePlate-Body.stl" scale="1.0 1.0 1.0"/>
+                <mesh filename="package://my_robot_description/mesh/CADv0/_mod_basePlate-Body.stl" scale="0.001 0.001 0.001"/>
             </geometry>
             <origin xyz="0 0 0" rpy="0 0 0"/>
-            <material name="white"/>
+            <material name="grey"/>
         </visual>
         <collision>
             <geometry>
-                <mesh filename="package://my_robot_description/mesh/CADv0/_mod_basePlate-Body.stl" scale="1.0 1.0 1.0"/>
+                <box size="0.132 0.096 0.004"/>
             </geometry>
-            <origin xyz="0 0 -0.002" rpy="0 0 0"/>
+            <origin xyz="0 -0.012 0.002" rpy="0 0 0"/>
         </collision>
         <xacro:lazy_inertia m="1.0"/>
@@ -28,14 +26,14 @@
         <visual>
             <geometry>
-                <mesh filename="package://my_robot_description/mesh/CADv0/_mod_XL-430holderBasic-Body.stl" scale="1.0 1.0 1.0"/>
+                <mesh filename="package://my_robot_description/mesh/CADv0/_mod_XL-430holderBasic-Body.stl" scale="0.001 0.001 0.001"/>
             </geometry>
-            <material name="grey"/>
-            <origin xyz="0 0 0" rpy="0 0 0"/>
+            <material name="white"/>
+            <origin xyz="0 0 0" rpy="0 0 ${urdf_pi/2}"/>
         </visual>
         <collision>
             <geometry>
-                <mesh filename="package://my_robot_description/mesh/CADv0/_mod_XL-430holderBasic-Body.stl" scale="1.0 1.0 1.0"/>
+                <box size="0.037 0.032 0.014"/>
             </geometry>
-            <origin xyz="0 0 -0.007" rpy="0 0 0"/>
+            <origin xyz="0 0 0.007" rpy="0 0 ${urdf_pi/2}"/>
         </collision>
         <xacro:box_inertia m="0.01" x="0.037" y="0.032" z="0.014" o_xyz="0 0 -0.01" o_rpy="0 0 0"/>
@@ -44,12 +42,12 @@
         <parent link="base_link"/>
         <child  link="servo1_holder"/>
-        <origin xyz="0 0 0" rpy="0 0 0"/>
+        <origin xyz="-0.050 0.018 0.004" rpy="0 0 0"/>
     </joint>
-    <!--link name="servo1">
+    <link name="servo1">
         <visual>
             <geometry>
                 <box size="${servo_x} ${servo_y} ${servo_z}"/>
             </geometry>
-            <origin xyz="0 0 0" rpy="0 0 0"/>
+            <origin xyz="0 0 ${servo_y/2}" rpy="${urdf_pi/2} 0 0"/>
             <material name="black"/>
         </visual>
@@ -58,5 +56,5 @@
                 <box size="${servo_x} ${servo_y} ${servo_z}"/>
             </geometry>
-            <origin xyz="0 0 0" rpy="0 0 0"/>
+            <origin xyz="0 0 ${servo_y/2}" rpy="${urdf_pi/2} 0 0"/>
         </collision>
         <xacro:box_inertia m="0.0572" x="${servo_x}" y="${servo_y}" z="${servo_z}" o_xyz="0 0 0" o_rpy="0 0 0"/>
@@ -65,5 +63,5 @@
         <parent link="servo1_holder"/>
         <child  link="servo1"/>
-        <origin xyz="0 0 0" rpy="0 0 0"/>
+        <origin xyz="0 0 0.008" rpy="0 0 0"/>
     </joint>
     <link name="servo1_padding">
@@ -72,5 +70,5 @@
                 <cylinder radius="0.011" length="0.004"/>
             </geometry>
-            <origin xyz="0 0 0" rpy="0 0 0"/>
+            <origin xyz="0 -0.002 0" rpy="${urdf_pi/2} 0 0"/>
             <material name="white"/>
         </visual>
@@ -79,15 +77,84 @@
                 <cylinder radius="0.011" length="0.004"/>
             </geometry>
-            <origin xyz="0 0 0" rpy="0 0 0"/>
+            <origin xyz="0 -0.002 0" rpy="${urdf_pi/2} 0 0"/>
         </collision>
         <xacro:cylinder_inertia m="0.001" r="0.011" l="0.004" o_xyz="0 0 0" o_rpy="0 0 0"/>
     </link>
-    <joint name="servo1_servo1_padding" type="continuous">
+    <joint name="servo1_servo1_padding" type="revolute">
         <parent link="servo1"/>
         <child  link="servo1_padding"/>
-        <origin xyz="0 0 0" rpy="0 0 0"/>
+        <origin xyz="0 ${-servo_z/2 - 0.002} 0.01125" rpy="0 0 0"/>
         <axis xyz="0 1 0"/>
+        <limit effort="1000.0" velocity="1.0" lower="${3*urdf_pi/4}" upper="${5*urdf_pi/4}"/>
+        <dynamics friction="0.05" damping="0.1"/>
     </joint>
-    < ============================ -->
+    <!-- ============================ -->
+    <link name="servo2_holder">
+        <visual>
+            <geometry>
+                <mesh filename="package://my_robot_description/mesh/CADv0/_mod_XL-430holderBasic-Body.stl" scale="0.001 0.001 0.001"/>
+            </geometry>
+            <material name="white"/>
+            <origin xyz="0 0 0" rpy="${urdf_pi/2} 0 0"/>
+        </visual>
+        <collision>
+            <geometry>
+                <box size="0.037 0.032 0.014"/>
+            </geometry>
+            <origin xyz="0 -0.007 0" rpy="${urdf_pi/2} 0 0"/>
+        </collision>
+        <xacro:box_inertia m="0.01" x="0.037" y="0.032" z="0.014" o_xyz="0 0 -0.01" o_rpy="0 0 0"/>
+    </link>
+    <joint name="base_link_servo2_holder" type="fixed">
+        <parent link="servo1_padding"/>
+        <child  link="servo2_holder"/>
+        <origin xyz="0 -0.004 0" rpy="0 0 0"/>
+    </joint>
+    <!--link name="servo2">
+        <visual>
+            <geometry>
+                <box size="${servo_x} ${servo_y} ${servo_z}"/>
+            </geometry>
+            <origin xyz="0 0 ${servo_y/2}" rpy="${urdf_pi/2} 0 0"/>
+            <material name="black"/>
+        </visual>
+        <collision>
+            <geometry>
+                <box size="${servo_x} ${servo_y} ${servo_z}"/>
+            </geometry>
+            <origin xyz="0 0 ${servo_y/2}" rpy="${urdf_pi/2} 0 0"/>
+        </collision>
+        <xacro:box_inertia m="0.0572" x="${servo_x}" y="${servo_y}" z="${servo_z}" o_xyz="0 0 0" o_rpy="0 0 0"/>
+    </link>
+    <joint name="servo2_holder_servo2" type="fixed">
+        <parent link="servo2_holder"/>
+        <child  link="servo2"/>
+        <origin xyz="0 0 0.008" rpy="0 0 0"/>
+    </joint>
+    <link name="servo2_padding">
+        <visual>
+            <geometry>
+                <cylinder radius="0.011" length="0.004"/>
+            </geometry>
+            <origin xyz="0 -0.002 0" rpy="${urdf_pi/2} 0 0"/>
+            <material name="white"/>
+        </visual>
+        <collision>
+            <geometry>
+                <cylinder radius="0.011" length="0.004"/>
+            </geometry>
+            <origin xyz="0 -0.002 0" rpy="${urdf_pi/2} 0 0"/>
+        </collision>
+        <xacro:cylinder_inertia m="0.001" r="0.011" l="0.004" o_xyz="0 0 0" o_rpy="0 0 0"/>
+    </link>
+    <joint name="servo2_servo2_padding" type="revolute">
+        <parent link="servo2"/>
+        <child  link="servo2_padding"/>
+        <origin xyz="0 ${-servo_z/2 - 0.002} 0.01125" rpy="0 0 0"/>
+        <axis xyz="0 1 0"/>
+        <limit effort="1000.0" velocity="1.0" lower="${3*urdf_pi/4}" upper="${5*urdf_pi/4}"/>
+        <dynamics friction="0.05" damping="0.1"/>
+    </joint-->
+    <!-- ============================ -->
 </robot>
 <!-- ================================================================================================================================== -->

Commit message: - adding peice in urdf up to thigh

File: src/my_robot_description/urdf/my_robot_leg.xacro (robot description, xacro)
@@ -111,10 +111,10 @@
         <origin xyz="0 -0.004 0" rpy="0 0 0"/>
     </joint>
-    <!--link name="servo2">
-        <visual>
-            <geometry>
-                <box size="${servo_x} ${servo_y} ${servo_z}"/>
-            </geometry>
-            <origin xyz="0 0 ${servo_y/2}" rpy="${urdf_pi/2} 0 0"/>
+    <link name="servo2">
+        <visual>
+            <geometry>
+                <box size="${servo_x} ${servo_y} ${servo_z}"/>
+            </geometry>
+            <origin xyz="0 ${-servo_y/2} 0" rpy="0 ${urdf_pi/2} 0"/>
             <material name="black"/>
         </visual>
@@ -123,5 +123,5 @@
                 <box size="${servo_x} ${servo_y} ${servo_z}"/>
             </geometry>
-            <origin xyz="0 0 ${servo_y/2}" rpy="${urdf_pi/2} 0 0"/>
+            <origin xyz="0 ${-servo_y/2} 0" rpy="0 ${urdf_pi/2} 0"/>
         </collision>
         <xacro:box_inertia m="0.0572" x="${servo_x}" y="${servo_y}" z="${servo_z}" o_xyz="0 0 0" o_rpy="0 0 0"/>
@@ -130,5 +130,5 @@
         <parent link="servo2_holder"/>
         <child  link="servo2"/>
-        <origin xyz="0 0 0.008" rpy="0 0 0"/>
+        <origin xyz="0 -0.008 0" rpy="0 0 0"/>
     </joint>
     <link name="servo2_padding">
@@ -137,12 +137,12 @@
                 <cylinder radius="0.011" length="0.004"/>
             </geometry>
-            <origin xyz="0 -0.002 0" rpy="${urdf_pi/2} 0 0"/>
-            <material name="white"/>
-        </visual>
-        <collision>
-            <geometry>
-                <cylinder radius="0.011" length="0.004"/>
-            </geometry>
-            <origin xyz="0 -0.002 0" rpy="${urdf_pi/2} 0 0"/>
+            <origin xyz="0.002 0 0" rpy="0 ${urdf_pi/2} 0"/>
+            <material name="white"/>
+        </visual>
+        <collision>
+            <geometry>
+                <cylinder radius="0.011" length="0.004"/>
+            </geometry>
+            <origin xyz="0.002 0 0" rpy="0 ${urdf_pi/2} 0"/>
         </collision>
         <xacro:cylinder_inertia m="0.001" r="0.011" l="0.004" o_xyz="0 0 0" o_rpy="0 0 0"/>
@@ -151,10 +151,73 @@
         <parent link="servo2"/>
         <child  link="servo2_padding"/>
-        <origin xyz="0 ${-servo_z/2 - 0.002} 0.01125" rpy="0 0 0"/>
-        <axis xyz="0 1 0"/>
+        <origin xyz="${servo_z/2 + 0.002} -0.03525 0" rpy="0 0 0"/>
+        <axis xyz="1 0 0"/>
         <limit effort="1000.0" velocity="1.0" lower="${3*urdf_pi/4}" upper="${5*urdf_pi/4}"/>
         <dynamics friction="0.05" damping="0.1"/>
-    </joint-->
+    </joint>
     <!-- ============================ -->
+    <link name="inner_thigh">
+        <visual>
+            <geometry>
+                <mesh filename="package://my_robot_description/mesh/CADv0/_mod_thighInner-Body.stl" scale="0.001 0.001 0.001"/>
+            </geometry>
+            <material name="blue"/>
+            <origin xyz="0 0 0" rpy="${-urdf_pi/2} 0 ${-urdf_pi/2}"/>
+        </visual>
+        <collision>
+            <geometry>
+                <box size="0.032 0.040 0.006"/>
+            </geometry>
+            <origin xyz="0.003 -0.016 0" rpy="${-urdf_pi/2} 0 ${-urdf_pi/2}"/>
+        </collision>
+        <xacro:box_inertia m="0.01" x="0.040" y="0.032" z="0.006" o_xyz="0 0 0" o_rpy="0 0 0"/>
+    </link>
+    <joint name="servo2_padding_inner_thigh" type="fixed">
+        <parent link="servo2_padding"/>
+        <child  link="inner_thigh"/>
+        <origin xyz="0.004 0.016 0" rpy="0 0 0"/>
+    </joint>
+    <link name="outer_thigh">
+        <visual>
+            <geometry>
+                <mesh filename="package://my_robot_description/mesh/CADv0/_mod_thighOuter-Body.stl" scale="0.001 0.001 0.001"/>
+            </geometry>
+            <material name="blue"/>
+            <origin xyz="0 0 0" rpy="${-urdf_pi/2} 0 ${-urdf_pi/2}"/>
+        </visual>
+        <collision>
+            <geometry>
+                <box size="0.110 0.040 0.006"/>
+            </geometry>
+            <origin xyz="0.003 -0.055 0" rpy="${-urdf_pi/2} 0 ${-urdf_pi/2}"/>
+        </collision>
+        <xacro:box_inertia m="0.01" x="0.040" y="0.032" z="0.006" o_xyz="0 0 0" o_rpy="0 0 0"/>
+    </link>
+    <joint name="inner_thigh_outer_thigh" type="fixed">
+        <parent link="inner_thigh"/>
+        <child  link="outer_thigh"/>
+        <origin xyz="0.028 0 0" rpy="0 0 0"/>
+    </joint>
+    <link name="servo3">
+        <visual>
+            <geometry>
+                <box size="${servo_x} ${servo_y} ${servo_z}"/>
+            </geometry>
+            <origin xyz="0 ${-servo_y/2} 0" rpy="0 ${urdf_pi/2} 0"/>
+            <material name="black"/>
+        </visual>
+        <collision>
+            <geometry>
+                <box size="${servo_x} ${servo_y} ${servo_z}"/>
+            </geometry>
+            <origin xyz="0 ${-servo_y/2} 0" rpy="0 ${urdf_pi/2} 0"/>
+        </collision>
+        <xacro:box_inertia m="0.0572" x="${servo_x}" y="${servo_y}" z="${servo_z}" o_xyz="0 0 0" o_rpy="0 0 0"/>
+    </link>
+    <joint name="outer_thigh_servo3" type="fixed">
+        <parent link="outer_thigh"/>
+        <child  link="servo3"/>
+        <origin xyz="0.010 -0.006 0" rpy="0 0 0"/>
+    </joint>
 </robot>
 <!-- ================================================================================================================================== -->
