Commit message: - the origin of the .stl part is important for the orientation in urdf - updating the moment of initial orientations in my_robot_leg.xacro

File: src/my_robot_description/urdf/my_robot_leg.xacro (robot description, xacro)
@@ -37,5 +37,5 @@
             <origin xyz="0 0 0.007" rpy="0 0 ${urdf_pi/2}"/>
         </collision>
-        <xacro:box_inertia m="0.01" x="0.037" y="0.032" z="0.014" o_xyz="0 0 -0.01" o_rpy="0 0 0"/>
+        <xacro:box_inertia m="0.01" x="0.037" y="0.032" z="0.014" o_xyz="0 0 0.007" o_rpy="0 0 ${urdf_pi/2}"/>
     </link>
     <joint name="base_link_servo1_holder" type="fixed">
@@ -58,5 +58,5 @@
             <origin xyz="0 0 ${servo_y/2}" rpy="${urdf_pi/2} 0 0"/>
         </collision>
-        <xacro:box_inertia m="0.0572" x="${servo_x}" y="${servo_y}" z="${servo_z}" o_xyz="0 0 0" o_rpy="0 0 0"/>
+        <xacro:box_inertia m="0.0572" x="${servo_x}" y="${servo_y}" z="${servo_z}" o_xyz="0 0 ${servo_y/2}" o_rpy="${urdf_pi/2} 0 0"/>
     </link>
     <joint name="servo1_holder_servo1" type="fixed">
@@ -79,5 +79,5 @@
             <origin xyz="0 -0.002 0" rpy="${urdf_pi/2} 0 0"/>
         </collision>
-        <xacro:cylinder_inertia m="0.001" r="0.011" l="0.004" o_xyz="0 0 0" o_rpy="0 0 0"/>
+        <xacro:cylinder_inertia m="0.001" r="0.011" l="0.004" o_xyz="0 -0.002 0" o_rpy="${urdf_pi/2} 0 0"/>
     </link>
     <joint name="servo1_servo1_padding" type="revolute">
@@ -104,5 +104,5 @@
             <origin xyz="0 -0.007 0" rpy="${urdf_pi/2} 0 0"/>
         </collision>
-        <xacro:box_inertia m="0.01" x="0.037" y="0.032" z="0.014" o_xyz="0 0 -0.01" o_rpy="0 0 0"/>
+        <xacro:box_inertia m="0.01" x="0.037" y="0.032" z="0.014" o_xyz="0 -0.007 0" o_rpy="${urdf_pi/2} 0 0"/>
     </link>
     <joint name="base_link_servo2_holder" type="fixed">
@@ -125,5 +125,5 @@
             <origin xyz="0 ${-servo_y/2} 0" rpy="0 ${urdf_pi/2} 0"/>
         </collision>
-        <xacro:box_inertia m="0.0572" x="${servo_x}" y="${servo_y}" z="${servo_z}" o_xyz="0 0 0" o_rpy="0 0 0"/>
+        <xacro:box_inertia m="0.0572" x="${servo_x}" y="${servo_y}" z="${servo_z}" o_xyz="0 ${-servo_y/2} 0" o_rpy="0 ${urdf_pi/2} 0"/>
     </link>
     <joint name="servo2_holder_servo2" type="fixed">
@@ -146,5 +146,5 @@
             <origin xyz="0.002 0 0" rpy="0 ${urdf_pi/2} 0"/>
         </collision>
-        <xacro:cylinder_inertia m="0.001" r="0.011" l="0.004" o_xyz="0 0 0" o_rpy="0 0 0"/>
+        <xacro:cylinder_inertia m="0.001" r="0.011" l="0.004" o_xyz="0.002 0 0" o_rpy="0 ${urdf_pi/2} 0"/>
     </link>
     <joint name="servo2_servo2_padding" type="revolute">
@@ -171,5 +171,5 @@
             <origin xyz="0.003 -0.016 0" rpy="${-urdf_pi/2} 0 ${-urdf_pi/2}"/>
         </collision>
-        <xacro:box_inertia m="0.01" x="0.040" y="0.032" z="0.006" o_xyz="0 0 0" o_rpy="0 0 0"/>
+        <xacro:box_inertia m="0.01" x="0.040" y="0.032" z="0.006" o_xyz="0.003 -0.016 0" o_rpy="${-urdf_pi/2} 0 ${-urdf_pi/2}"/>
     </link>
     <joint name="servo2_padding_inner_thigh" type="fixed">
@@ -192,5 +192,5 @@
             <origin xyz="0.003 -0.055 0" rpy="${-urdf_pi/2} 0 ${-urdf_pi/2}"/>
         </collision>
-        <xacro:box_inertia m="0.01" x="0.040" y="0.032" z="0.006" o_xyz="0 0 0" o_rpy="0 0 0"/>
+        <xacro:box_inertia m="0.02" x="0.040" y="0.032" z="0.006" o_xyz="0.003 -0.055 0" o_rpy="${-urdf_pi/2} 0 ${-urdf_pi/2}"/>
     </link>
     <joint name="inner_thigh_outer_thigh" type="fixed">
@@ -213,5 +213,5 @@
             <origin xyz="0 ${-servo_y/2} 0" rpy="0 ${urdf_pi/2} 0"/>
         </collision>
-        <xacro:box_inertia m="0.0572" x="${servo_x}" y="${servo_y}" z="${servo_z}" o_xyz="0 0 0" o_rpy="0 0 0"/>
+        <xacro:box_inertia m="0.0572" x="${servo_x}" y="${servo_y}" z="${servo_z}" o_xyz="0 ${-servo_y/2} 0" o_rpy="0 ${urdf_pi/2} 0"/>
     </link>
     <joint name="outer_thigh_servo3" type="fixed">
@@ -232,7 +232,7 @@
                 <cylinder radius="0.011" length="0.006"/>
             </geometry>
-            <origin xyz="0 0 0" rpy="0 0 0"/>
-        </collision>
-        <xacro:cylinder_inertia m="0.001" r="0.011" l="0.006" o_xyz="0 0 0" o_rpy="0 0 0"/>
+            <origin xyz="0 0 0" rpy="${-urdf_pi/2} 0 ${urdf_pi/2}"/>
+        </collision>
+        <xacro:cylinder_inertia m="0.001" r="0.011" l="0.006" o_xyz="0 0 0" o_rpy="${-urdf_pi/2} 0 ${urdf_pi/2}"/>
     </link>
     <joint name="servo3_calfJoint" type="revolute">
@@ -241,5 +241,5 @@
         <origin xyz="${-servo_z/2-0.0025-0.002} ${-0.011-0.010-0.0025/2} 0" rpy="0 0 0"/>
         <axis xyz="1 0 0"/>
-        <limit effort="1000.0" velocity="1.0" lower="0" upper="${2*urdf_pi}"/>
+        <limit effort="1000.0" velocity="1.0" lower="${3*urdf_pi/4}" upper="${5*urdf_pi/4}"/>
         <dynamics friction="0.05" damping="0.1"/>
     </joint>
@@ -258,10 +258,14 @@
             <origin xyz="0.003 -0.055 0" rpy="0 0 0"/>
         </collision>
-        <xacro:box_inertia m="0.01" x="0.040" y="0.032" z="0.006" o_xyz="0 0 0" o_rpy="0 0 0"/>
-    </link>
-    <joint name="calfJoint_calfFeet" type="fixed">
-        <parent link="calfJoint"/>
+        <xacro:box_inertia m="0.02" x="0.040" y="0.032" z="0.006" o_xyz="0 0 0" o_rpy="0 0 0"/>
+    </link>
+    <joint name="servo3_calfFeet" type="revolute">
+        <parent link="servo3"/>
         <child  link="calfFeet"/>
         <origin xyz="-0.0025 ${-0.09+0.011+0.010+0.0025/2} -0.032" rpy="0 0 0"/>
+        <axis xyz="1 0 0"/>
+        <mimic joint="servo3_calfJoint" multiplier="1.0" offset="0.0"/>
+        <limit effort="1000.0" velocity="1.0" lower="${3*urdf_pi/4}" upper="${5*urdf_pi/4}"/>
+        <dynamics friction="0.05" damping="0.1"/>
     </joint>
 </robot>

Commit message: - correct the geometry, the feet was pointing at the opposite direction

File: src/my_robot_description/urdf/my_robot_leg.xacro (robot description, xacro)
@@ -22,5 +22,5 @@
         <xacro:lazy_inertia m="1.0"/>
     </link>
-    <!-- ============================ -->
+    <!-- ============================================================================================================================== -->
     <link name="servo1_holder">
         <visual>
@@ -89,5 +89,5 @@
         <dynamics friction="0.05" damping="0.1"/>
     </joint>
-    <!-- ============================ -->
+    <!-- ============================================================================================================================== -->
     <link name="servo2_holder">
         <visual>
@@ -156,5 +156,5 @@
         <dynamics friction="0.05" damping="0.1"/>
     </joint>
-    <!-- ============================ -->
+    <!-- ============================================================================================================================== -->
     <link name="inner_thigh">
         <visual>
@@ -225,5 +225,5 @@
                 <mesh filename="package://my_robot_description/mesh/CADv0/_mod_calfJoint-Body.stl" scale="0.001 0.001 0.001"/>
             </geometry>
-            <origin xyz="0 0 0" rpy="${-urdf_pi/2} 0 ${urdf_pi/2}"/>
+            <origin xyz="0 0 0" rpy="${urdf_pi/2} 0 ${-urdf_pi/2}"/>
             <material name="white"/>
         </visual>
@@ -232,7 +232,7 @@
                 <box size="0.022 0.051 0.0065"/>
             </geometry>
-            <origin xyz="-0.0005 0 -0.0145" rpy="${-urdf_pi/2} 0 ${urdf_pi/2}"/>
-        </collision>
-        <xacro:box_inertia m="0.0015" x="0.022" y="0.051" z="0.0065" o_xyz="-0.0005 0 -0.0145" o_rpy="${-urdf_pi/2} 0 ${urdf_pi/2}"/>
+            <origin xyz="-0.0005 0 0.0145" rpy="${urdf_pi/2} 0 ${-urdf_pi/2}"/>
+        </collision>
+        <xacro:box_inertia m="0.0015" x="0.022" y="0.051" z="0.0065" o_xyz="-0.0005 0 0.0145" o_rpy="${urdf_pi/2} 0 ${-urdf_pi/2}"/>
     </link>
     <joint name="servo3_calfJoint" type="revolute">
@@ -250,5 +250,5 @@
             </geometry>
             <material name="purple"/>
-            <origin xyz="0 -0.008 -0.035" rpy="0 ${-urdf_pi/2} 0"/>
+            <origin xyz="-0.004 -0.008 0.035" rpy="0 ${urdf_pi/2} 0"/>
         </visual>
         <collision>
@@ -256,12 +256,13 @@
                 <box size="0.150 0.016 0.004"/>
             </geometry>
-            <origin xyz="-0.002 ${-0.008+0.008} ${-0.035+0.080}" rpy="0 ${-urdf_pi/2} 0"/>
-        </collision>
-        <xacro:box_inertia m="0.02" x="0.150" y="0.016" z="0.004" o_xyz="${-servo_z/2-0.002-0.0025-0.002} ${-0.008+0.008} ${-0.035+0.080}" o_rpy="0 ${-urdf_pi/2} 0"/>
+            <origin xyz="-0.002 ${-0.008+0.008} ${0.035-0.080}" rpy="0 ${-urdf_pi/2} 0"/>
+        </collision>
+        <xacro:box_inertia m="0.02" x="0.150" y="0.016" z="0.004"
+                           o_xyz="${-servo_z/2-0.002-0.0025-0.002} ${-0.008+0.008} ${0.035-0.080}" o_rpy="0 ${-urdf_pi/2} 0"/>
     </link>
     <joint name="servo3_calfFeet" type="revolute">
         <parent link="servo3"/>
         <child  link="calfFeet"/>
-        <origin xyz="${-servo_z/2-0.002-0.0025} -0.101 0" rpy="0 0 0"/>
+        <origin xyz="${-servo_z/2-0.002-0.0025} ${-0.101+0.004} 0" rpy="0 0 0"/>
         <axis xyz="1 0 0"/>
         <mimic joint="servo3_calfJoint" multiplier="1.0" offset="0.0"/>
@@ -288,5 +289,5 @@
         <parent link="calfFeet"/>
         <child  link="calfSphere"/>
-        <origin xyz="-0.002 0.004 ${0.150-0.035}" rpy="0 0 0"/>
+        <origin xyz="-0.002 0.004 ${-0.150+0.035}" rpy="0 0 0"/>
     </joint>
 </robot>

Commit message: - lifting up the base main_board to avoid collision with ground + update collision geometry to sustain the T shape

File: src/my_robot_description/urdf/my_robot_leg.xacro (robot description, xacro)
@@ -9,4 +9,20 @@
         <visual>
             <geometry>
+                <box size="0.052 0.096 0.06"/>
+            </geometry>
+            <origin xyz="0 0 -0.03" rpy="0 0 0"/>
+            <material name="grey"/>
+        </visual>
+        <collision>
+            <geometry>
+                <box size="0.052 0.096 0.06"/>
+            </geometry>
+            <origin xyz="0 0 -0.03" rpy="0 0 0"/>
+        </collision>
+        <xacro:lazy_inertia m="10.0"/>
+    </link>
+    <link name="main_board">
+        <visual>
+            <geometry>
                 <mesh filename="package://my_robot_description/mesh/CADv0/_mod_basePlate-Body.stl" scale="0.001 0.001 0.001"/>
             </geometry>
@@ -16,10 +32,15 @@
         <collision>
             <geometry>
-                <box size="0.132 0.096 0.004"/>
-            </geometry>
-            <origin xyz="0 -0.012 0.002" rpy="0 0 0"/>
+                <box size="0.132 0.036 0.004"/>
+            </geometry>
+            <origin xyz="0 0.018 0.002" rpy="0 0 0"/>
         </collision>
         <xacro:lazy_inertia m="1.0"/>
     </link>
+    <joint name="base_link_main_board" type="fixed">
+        <parent link="base_link"/>
+        <child  link="main_board"/>
+        <origin xyz="0 0.012 -0.004" rpy="0 0 0"/>
+    </joint>
     <!-- ============================================================================================================================== -->
     <link name="servo1_holder">
@@ -39,6 +60,6 @@
         <xacro:box_inertia m="0.01" x="0.037" y="0.032" z="0.014" o_xyz="0 0 0.007" o_rpy="0 0 ${urdf_pi/2}"/>
     </link>
-    <joint name="base_link_servo1_holder" type="fixed">
-        <parent link="base_link"/>
+    <joint name="main_board_servo1_holder" type="fixed">
+        <parent link="main_board"/>
         <child  link="servo1_holder"/>
         <origin xyz="-0.050 0.018 0.004" rpy="0 0 0"/>

Commit message: - update the angle range to support initial angle of 0 degrees

File: src/my_robot_description/urdf/my_robot_leg.xacro (robot description, xacro)
@@ -107,5 +107,5 @@
         <origin xyz="0 ${-servo_z/2-0.002} ${0.01+0.0025/2}" rpy="0 0 0"/>
         <axis xyz="0 1 0"/>
-        <limit effort="1000.0" velocity="1.0" lower="${3*urdf_pi/4}" upper="${5*urdf_pi/4}"/>
+        <limit effort="1000.0" velocity="1.0" lower="${-2*urdf_pi/8}" upper="${2*urdf_pi/8}"/>
         <dynamics friction="0.05" damping="0.1"/>
     </joint>
@@ -174,5 +174,5 @@
         <origin xyz="${servo_z/2+0.002} -0.03525 0" rpy="0 0 0"/>
         <axis xyz="1 0 0"/>
-        <limit effort="1000.0" velocity="1.0" lower="${3*urdf_pi/4}" upper="${5*urdf_pi/4}"/>
+        <limit effort="1000.0" velocity="1.0" lower="${-2*urdf_pi/8}" upper="${2*urdf_pi/8}"/>
         <dynamics friction="0.05" damping="0.1"/>
     </joint>
@@ -262,5 +262,5 @@
         <origin xyz="${-servo_z/2-0.002-0.0025} ${-0.01-0.0025/2} 0" rpy="0 0 0"/>
         <axis xyz="1 0 0"/>
-        <limit effort="1000.0" velocity="1.0" lower="${5*urdf_pi/8}" upper="${11*urdf_pi/8}"/>
+        <limit effort="1000.0" velocity="1.0" lower="${-3*urdf_pi/8}" upper="${3*urdf_pi/8}"/>
         <dynamics friction="0.05" damping="0.1"/>
     </joint>
@@ -288,5 +288,5 @@
         <axis xyz="1 0 0"/>
         <mimic joint="servo3_calfJoint" multiplier="1.0" offset="0.0"/>
-        <limit effort="1000.0" velocity="1.0" lower="${5*urdf_pi/8}" upper="${11*urdf_pi/8}"/>
+        <limit effort="1000.0" velocity="1.0" lower="${-3*urdf_pi/8}" upper="${3*urdf_pi/8}"/>
         <dynamics friction="0.05" damping="0.1"/>
     </joint>

Commit message: - initial setup of moveit2 with assistance

File: src/my_robot_description/urdf/my_robot_leg.xacro (robot description, xacro)
@@ -107,5 +107,5 @@
         <origin xyz="0 ${-servo_z/2-0.002} ${0.01+0.0025/2}" rpy="0 0 0"/>
         <axis xyz="0 1 0"/>
-        <limit effort="1000.0" velocity="1.0" lower="${-2*urdf_pi/8}" upper="${2*urdf_pi/8}"/>
+        <limit effort="1000.0" velocity="1.0" lower="${6*urdf_pi/8}" upper="${10*urdf_pi/8}"/>
         <dynamics friction="0.05" damping="0.1"/>
     </joint>
@@ -174,5 +174,5 @@
         <origin xyz="${servo_z/2+0.002} -0.03525 0" rpy="0 0 0"/>
         <axis xyz="1 0 0"/>
-        <limit effort="1000.0" velocity="1.0" lower="${-2*urdf_pi/8}" upper="${2*urdf_pi/8}"/>
+        <limit effort="1000.0" velocity="1.0" lower="${6*urdf_pi/8}" upper="${10*urdf_pi/8}"/>
         <dynamics friction="0.05" damping="0.1"/>
     </joint>
@@ -262,5 +262,5 @@
         <origin xyz="${-servo_z/2-0.002-0.0025} ${-0.01-0.0025/2} 0" rpy="0 0 0"/>
         <axis xyz="1 0 0"/>
-        <limit effort="1000.0" velocity="1.0" lower="${-3*urdf_pi/8}" upper="${3*urdf_pi/8}"/>
+        <limit effort="1000.0" velocity="1.0" lower="${5*urdf_pi/8}" upper="${11*urdf_pi/8}"/>
         <dynamics friction="0.05" damping="0.1"/>
     </joint>
@@ -288,5 +288,5 @@
         <axis xyz="1 0 0"/>
         <mimic joint="servo3_calfJoint" multiplier="1.0" offset="0.0"/>
-        <limit effort="1000.0" velocity="1.0" lower="${-3*urdf_pi/8}" upper="${3*urdf_pi/8}"/>
+        <limit effort="1000.0" velocity="1.0" lower="${5*urdf_pi/8}" upper="${11*urdf_pi/8}"/>
         <dynamics friction="0.05" damping="0.1"/>
     </joint>

Commit message: - editing to allow moveit to control the tip of the feet "calfSphere" without using end effector. Instead use the chain instead of joint option in src/my_robot_moveit_config/config/my_robot.srdf

File: src/my_robot_description/urdf/my_robot_leg.xacro (robot description, xacro)
@@ -241,4 +241,29 @@
         <origin xyz="${servo_y/2-0.006-0.0025} -0.004 0" rpy="0 0 0"/>
     </joint>
+    <link name="calfFeet">
+        <visual>
+            <geometry>
+                <mesh filename="package://my_robot_description/mesh/CADv0/calfFeet-Body.stl" scale="0.001 0.001 0.001"/>
+            </geometry>
+            <material name="purple"/>
+            <origin xyz="-0.004 -0.008 0.035" rpy="0 ${urdf_pi/2} 0"/>
+        </visual>
+        <collision>
+            <geometry>
+                <box size="0.150 0.016 0.004"/>
+            </geometry>
+            <origin xyz="-0.002 ${-0.008+0.008} ${0.035-0.080}" rpy="0 ${-urdf_pi/2} 0"/>
+        </collision>
+        <xacro:box_inertia m="0.02" x="0.150" y="0.016" z="0.004"
+                           o_xyz="${-servo_z/2-0.002-0.0025-0.002} ${-0.008+0.008} ${0.035-0.080}" o_rpy="0 ${-urdf_pi/2} 0"/>
+    </link>
+    <joint name="servo3_calfFeet" type="revolute">
+        <parent link="servo3"/>
+        <child  link="calfFeet"/>
+        <origin xyz="${-servo_z/2-0.002-0.0025} ${-0.101+0.004} 0" rpy="0 0 0"/>
+        <axis xyz="1 0 0"/>
+        <limit effort="1000.0" velocity="1.0" lower="${5*urdf_pi/8}" upper="${11*urdf_pi/8}"/>
+        <dynamics friction="0.05" damping="0.1"/>
+    </joint>
     <link name="calfJoint">
         <visual>
@@ -262,30 +287,5 @@
         <origin xyz="${-servo_z/2-0.002-0.0025} ${-0.01-0.0025/2} 0" rpy="0 0 0"/>
         <axis xyz="1 0 0"/>
-        <limit effort="1000.0" velocity="1.0" lower="${5*urdf_pi/8}" upper="${11*urdf_pi/8}"/>
-        <dynamics friction="0.05" damping="0.1"/>
-    </joint>
-    <link name="calfFeet">
-        <visual>
-            <geometry>
-                <mesh filename="package://my_robot_description/mesh/CADv0/calfFeet-Body.stl" scale="0.001 0.001 0.001"/>
-            </geometry>
-            <material name="purple"/>
-            <origin xyz="-0.004 -0.008 0.035" rpy="0 ${urdf_pi/2} 0"/>
-        </visual>
-        <collision>
-            <geometry>
-                <box size="0.150 0.016 0.004"/>
-            </geometry>
-            <origin xyz="-0.002 ${-0.008+0.008} ${0.035-0.080}" rpy="0 ${-urdf_pi/2} 0"/>
-        </collision>
-        <xacro:box_inertia m="0.02" x="0.150" y="0.016" z="0.004"
-                           o_xyz="${-servo_z/2-0.002-0.0025-0.002} ${-0.008+0.008} ${0.035-0.080}" o_rpy="0 ${-urdf_pi/2} 0"/>
-    </link>
-    <joint name="servo3_calfFeet" type="revolute">
-        <parent link="servo3"/>
-        <child  link="calfFeet"/>
-        <origin xyz="${-servo_z/2-0.002-0.0025} ${-0.101+0.004} 0" rpy="0 0 0"/>
-        <axis xyz="1 0 0"/>
-        <mimic joint="servo3_calfJoint" multiplier="1.0" offset="0.0"/>
+        <mimic joint="servo3_calfFeet" multiplier="1.0" offset="0.0"/>
         <limit effort="1000.0" velocity="1.0" lower="${5*urdf_pi/8}" upper="${11*urdf_pi/8}"/>
         <dynamics friction="0.05" damping="0.1"/>

File: src/my_robot_moveit_config/config/my_robot.ros2_control.xacro (robot description, xacro)
@@ -20,8 +20,8 @@
                 </state_interface>
             </joint>
-            <joint name="servo3_calfJoint">
+            <joint name="servo3_calfFeet">
                 <command_interface name="position"/>
                 <state_interface name="position">
-                  <param name="initial_value">${initial_positions['servo3_calfJoint']}</param>
+                  <param name="initial_value">${initial_positions['servo3_calfFeet']}</param>
                 </state_interface>
             </joint>

Commit message: - problem syncing moveit and joint_state_broadcaster, gemini states: ros2 topic hz /joint_states If it is lower than 10Hz, MoveIt will often throw the "recent timestamp" error. You should aim for 30Hz to 50Hz. - need to optimize hardware_interface_my_robot_dynamixel_u2d2_xl430.cpp

File: src/my_robot_description/urdf/my_robot_leg.xacro (robot description, xacro)
@@ -6,4 +6,5 @@
     <xacro:property name="servo_z" value="0.034"/>
 <!-- ================================================================================================================================== -->
+    <link name="world"/>
     <link name="base_link">
         <visual>
@@ -22,4 +23,8 @@
         <xacro:lazy_inertia m="10.0"/>
     </link>
+    <joint name="world_base_link" type="fixed">
+        <parent link="world"/>
+        <child link="base_link"/>
+    </joint>
     <link name="main_board">
         <visual>

Commit message: - now my_robot.with_commander.launch.py loads actual moveit config, IK now available. - improving revolution limits for my_robot_leg.xacro

File: src/my_robot_description/urdf/my_robot_leg.xacro (robot description, xacro)
@@ -111,6 +111,6 @@
         <child  link="servo1_padding"/>
         <origin xyz="0 ${-servo_z/2-0.002} ${0.01+0.0025/2}" rpy="0 0 0"/>
-        <axis xyz="0 1 0"/>
-        <limit effort="1000.0" velocity="1.0" lower="${6*urdf_pi/8}" upper="${10*urdf_pi/8}"/>
+        <axis xyz="0 -1 0"/>
+        <limit effort="1000.0" velocity="1.0" lower="2.5" upper="4.0"/>
         <dynamics friction="0.05" damping="0.1"/>
     </joint>
@@ -179,5 +179,5 @@
         <origin xyz="${servo_z/2+0.002} -0.03525 0" rpy="0 0 0"/>
         <axis xyz="1 0 0"/>
-        <limit effort="1000.0" velocity="1.0" lower="${6*urdf_pi/8}" upper="${10*urdf_pi/8}"/>
+        <limit effort="1000.0" velocity="1.0" lower="2.0" upper="4.0"/>
         <dynamics friction="0.05" damping="0.1"/>
     </joint>
@@ -267,6 +267,6 @@
         <child  link="calfFeet"/>
         <origin xyz="${-servo_z/2-0.002-0.0025} ${-0.101+0.004} 0" rpy="0 0 0"/>
-        <axis xyz="1 0 0"/>
-        <limit effort="1000.0" velocity="1.0" lower="${5*urdf_pi/8}" upper="${11*urdf_pi/8}"/>
+        <axis xyz="-1 0 0"/>
+        <limit effort="1000.0" velocity="1.0" lower="2.0" upper="4.0"/>
         <dynamics friction="0.05" damping="0.1"/>
     </joint>

Commit message: - resolved the [move_group.moveit.moveit.core.conversions]: Found empty JointState message problem - pilz linear motion now available! Do remember to move to the starting post first though

File: src/my_robot_description/urdf/my_robot_leg.xacro (robot description, xacro)
@@ -289,17 +289,12 @@
                            o_xyz="-0.0005 0 0.0145" o_rpy="${urdf_pi/2} 0 ${-urdf_pi/2}"/>
     </link>
-    <!--joint name="servo3_calfJoint" type="revolute">
+    <joint name="servo3_calfJoint" type="revolute">
         <parent link="servo3"/>
         <child  link="calfJoint"/>
         <origin xyz="${-servo_z/2-0.002-0.0025} ${-0.01-0.0025/2} 0" rpy="0 0 0"/>
-        <axis xyz="1 0 0"/>
+        <axis xyz="-1 0 0"/>
         <mimic joint="servo3_calfFeet" multiplier="1.0" offset="0.0"/>
         <limit effort="1000.0" velocity="1.0" lower="${5*urdf_pi/8}" upper="${11*urdf_pi/8}"/>
         <dynamics friction="0.05" damping="0.1"/>
-    </joint-->
-    <joint name="servo3_calfJoint" type="fixed">
-        <parent link="servo3"/>
-        <child  link="calfJoint"/>
-        <origin xyz="${-servo_z/2-0.002-0.0025} ${-0.01-0.0025/2} 0" rpy="0 0 0"/>
     </joint>
     <link name="calfSphere">
