Commit message: - trying to debug TOTG - also ros2 param list seems to hang

File: src/my_robot_description/urdf/my_robot_leg.xacro (robot description, xacro)
@@ -112,5 +112,5 @@
         <origin xyz="0 ${-servo_z/2-0.002} ${0.01+0.0025/2}" rpy="0 0 0"/>
         <axis xyz="0 -1 0"/>
-        <limit effort="1000.0" velocity="1.0" lower="2.5" upper="4.0"/>
+        <limit effort="1000.0" velocity="20.0" lower="2.5" upper="4.0"/>
         <dynamics friction="0.05" damping="0.1"/>
     </joint>
@@ -179,5 +179,5 @@
         <origin xyz="${servo_z/2+0.002} -0.03525 0" rpy="0 0 0"/>
         <axis xyz="1 0 0"/>
-        <limit effort="1000.0" velocity="1.0" lower="2.0" upper="4.0"/>
+        <limit effort="1000.0" velocity="20.0" lower="2.0" upper="4.0"/>
         <dynamics friction="0.05" damping="0.1"/>
     </joint>
@@ -269,5 +269,5 @@
         <origin xyz="${-servo_z/2-0.002-0.0025} ${-0.101+0.004} 0" rpy="0 0 0"/>
         <axis xyz="-1 0 0"/>
-        <limit effort="1000.0" velocity="1.0" lower="2.0" upper="4.0"/>
+        <limit effort="1000.0" velocity="20.0" lower="2.0" upper="4.0"/>
         <dynamics friction="0.05" damping="0.1"/>
     </joint>
@@ -295,5 +295,5 @@
         <axis xyz="-1 0 0"/>
         <mimic joint="servo3_calfFeet" multiplier="1.0" offset="0.0"/>
-        <limit effort="1000.0" velocity="1.0" lower="${5*urdf_pi/8}" upper="${11*urdf_pi/8}"/>
+        <limit effort="1000.0" velocity="20.0" lower="${5*urdf_pi/8}" upper="${11*urdf_pi/8}"/>
         <dynamics friction="0.05" damping="0.1"/>
     </joint>
