Commit message: - resolve the radiant to dxl resolution convertion range/type issue. - set the servos only on joint1, joint4, and joint6 that have -pi to pi range

File: src/my_robot_description/urdf/common_properties.xacro (robot description, xacro)
@@ -1,4 +1,5 @@
 <?xml version="1.0"?>
 <robot xmlns:xacro="http://www.ros.org/wiki/xacro">
+    <xacro:property name="urdf_pi" value="3.14159"/>
     <material name="grey">
         <color rgba="0.5 0.5 0.5 1"/>

File: src/my_robot_description/urdf/ma_robot.ros2_control.xacro (robot description, xacro)
@@ -6,6 +6,6 @@
             <plugin>ma_robot_namespace/HardwareInterfaceU2D2_ma_robot</plugin>
             <param name="joint1_servo_channel">11</param>
-            <param name="joint2_servo_channel">12</param>
-            <param name="joint3_servo_channel">13</param>
+            <param name="joint4_servo_channel">12</param>
+            <param name="joint6_servo_channel">13</param>
         </hardware>
         <joint name="joint1">

File: src/my_robot_description/urdf/ma_robot_arm.xacro (robot description, xacro)
@@ -126,5 +126,5 @@
         <origin xyz="0 0 0.1" rpy="0 0 0" />
         <axis xyz="0 0 1" />
-        <limit effort="1000.0" velocity="1.0" lower="-3.14" upper="3.14" />
+        <limit effort="1000.0" velocity="1.0" lower="${-urdf_pi}" upper="${urdf_pi}" />
         <dynamics friction="0.05" damping="0.1" />
     </joint>
@@ -150,5 +150,5 @@
         <origin xyz="0 0 0.1" rpy="0 0 0" />
         <axis xyz="0 0 1" />
-        <limit effort="1000.0" velocity="1.0" lower="-3.14" upper="3.14" />
+        <limit effort="1000.0" velocity="1.0" lower="${-urdf_pi}" upper="${urdf_pi}" />
         <dynamics friction="0.05" damping="0.1" />
     </joint>
@@ -158,5 +158,5 @@
         <origin xyz="0 0 0.5" rpy="0 0 0" />
         <axis xyz="0 1 0" />
-        <limit effort="1000.0" velocity="1.0" lower="-1.57" upper="1.57" />
+        <limit effort="1000.0" velocity="1.0" lower="${-urdf_pi/2.0}" upper="${urdf_pi/2.0}" />
         <dynamics friction="0.05" damping="0.1" />
     </joint>
@@ -166,5 +166,5 @@
         <origin xyz="0 0 0.05" rpy="0 0 0" />
         <axis xyz="0 0 1" />
-        <limit effort="1000.0" velocity="1.0" lower="-3.14" upper="3.14" />
+        <limit effort="1000.0" velocity="1.0" lower="${-urdf_pi}" upper="${urdf_pi}" />
         <dynamics friction="0.05" damping="0.1" />
     </joint>

Commit message: - initial urdf for 1 leg, need actual rvis to determine the final positioning

File: src/my_robot_description/urdf/common_properties.xacro (robot description, xacro)
@@ -2,4 +2,10 @@
 <robot xmlns:xacro="http://www.ros.org/wiki/xacro">
     <xacro:property name="urdf_pi" value="3.14159"/>
+    <material name="white">
+        <color rgba="1 1 1 1"/>
+    </material>
+    <material name="black">
+        <color rgba="0 0 0 1"/>
+    </material>
     <material name="grey">
         <color rgba="0.5 0.5 0.5 1"/>

File: src/my_robot_description/urdf/my_robot_leg.xacro (robot description, xacro)
@@ -1,36 +1,96 @@
 <?xml version="1.0"?>
-<!-- ======================================================================================================== -->
-<!-- reference from  Antonio Brandi, "Robotics and ROS 2 - Learn by Doing! Manipulators" (Udemy) -->
+<!-- ================================================================================================================================== -->
 <robot xmlns:xacro="http://www.ros.org/wiki/xacro" name="my_robot_leg">
     <xacro:include filename="$(find my_robot_description)/urdf/common_properties.xacro"/>
-    <!-- xacro:include filename="$(find robot_build)/urdf/arduinobot.ros2_control.xacro"/-->
-    <xacro:property name="effort"   value="30.0" />
-    <xacro:property name="velocity" value="10.0" />
-<!-- ======================================================================================================== -->
-    <!-- Links -->
+    <xacro:property name="effort"   value="30.0"/>
+    <xacro:property name="velocity" value="10.0"/>
+    <xacro:property name="servo_x" value="0.0285"/>
+    <xacro:property name="servo_y" value="0.0465"/>
+    <xacro:property name="servo_z" value="0.034"/>
+<!-- ================================================================================================================================== -->
     <link name="world"/>
+    <!-- ============================ -->
     <link name="base_link">
         <visual>
-            <origin rpy="0 0 0" xyz="-0.5 -0.5 0"/>
             <geometry>
-                <mesh filename="package://my_robot_description/mesh/CADv0/basePlate-Body.stl" scale="0.01 0.01 0.01"/>
+                <mesh filename="package://my_robot_description/mesh/CADv0/_mod_basePlate-Body.stl" scale="1.0 1.0 1.0"/>
             </geometry>
-            <material name="red"/>
+            <origin rpy="0 0 0" xyz="0 0 0"/>
+            <material name="white"/>
         </visual>
         <collision>
-            <origin rpy="0 0 0" xyz="-0.5 -0.5 0"/>
             <geometry>
-                <mesh filename="package://my_robot_description/mesh/CADv0/basePlate-Body.stl" scale="0.01 0.01 0.01"/>
+                <mesh filename="package://my_robot_description/mesh/CADv0/_mod_basePlate-Body.stl" scale="1.0 1.0 1.0"/>
             </geometry>
+            <origin rpy="0 0 0" xyz="0 0 0"/>
         </collision>
         <xacro:lazy_inertia m="1.0"/>
     </link>
-<!-- ======================================================================================================== -->
-    <!-- Joints -->
-    <joint name="virtual_joint" type="fixed">
-        <parent link="world"/>
-        <child link="base_link"/>
+    <!-- ============================ -->
+    <link name="servo1_holder">
+        <visual>
+            <geometry>
+                <mesh filename="package://my_robot_description/mesh/CADv0/_mod_XL-430holderBasic.stl" scale="1.0 1.0 1.0"/>
+            </geometry>
+            <material name="grey"/>
+            <origin rpy="0 0 0" xyz="0 0 0"/>
+        </visual>
+        <collision>
+            <geometry>
+                <mesh filename="package://my_robot_description/mesh/CADv0/_mod_XL-430holderBasic.stl" scale="1.0 1.0 1.0"/>
+            </geometry>
+            <origin rpy="0 0 0" xyz="0 0 0"/>
+        </collision>
+        <xacro:box_inertia m="0.01" x="0.037" y="0.032" z="0.014" o_xyz="0 0 -0.01" o_rpy="0 0 0"/>
+    </link>
+    <joint name="base_link_servo1_holder" type="fixed">
+        <parent link="base_link"/>
+        <child  link="servo1_holder"/>
+        <origin xyz="0 0 0.004" rpy="0 0 0"/>
+    </joint>
+    <link name="servo1">
+        <visual>
+            <geometry>
+                <box size="${servo_x} ${servo_y} ${servo_z}"/>
+            </geometry>
+            <origin xyz="0 0 0" rpy="0 0 0"/>
+            <material name="black"/>
+        </visual>
+        <collision>
+            <geometry>
+                <box size="${servo_x} ${servo_y} ${servo_z}"/>
+            </geometry>
+            <origin rpy="0 0 0" xyz="0 0 0"/>
+        </collision>
+        <xacro:box_inertia m="0.0572" x="${servo_x}" y="${servo_y}" z="${servo_z}" o_xyz="0 0 0" o_rpy="0 0 0"/>
+    </link>
+    <joint name="servo1_holder_servo1" type="fixed">
+        <parent link="servo1_holder"/>
+        <child  link="servo1"/>
         <origin xyz="0 0 0" rpy="0 0 0"/>
     </joint>
-<!-- ======================================================================================================== -->
+    <link name="servo1_padding">
+        <visual>
+            <geometry>
+                <cylinder radius="0.011" length="0.004"/>
+            </geometry>
+            <origin xyz="0 0 0" rpy="0 0 0"/>
+            <material name="white"/>
+        </visual>
+        <collision>
+            <geometry>
+                <cylinder radius="0.011" length="0.004"/>
+            </geometry>
+            <origin rpy="0 0 0" xyz="0 0 0"/>
+        </collision>
+        <xacro:cylinder_inertia m="0.001" x="0.011" l="0.004" o_xyz="0 0 0" o_rpy="0 0 0"/>
+    </link>
+    <joint name="servo1_servo1_padding" type="continuous">
+        <parent link="servo1"/>
+        <child  link="servo1_padding"/>
+        <origin xyz="0 0 0" rpy="0 0 0"/>
+        <axis xyz="0 1 0"/>
+    </joint>
+    <!-- ============================ -->
 </robot>
+<!-- ================================================================================================================================== -->

Commit message: - adding all the relevant peice in urdf, but much details still need update

File: src/my_robot_description/urdf/common_properties.xacro (robot description, xacro)
@@ -25,4 +25,7 @@
     <material name="yellow">
         <color rgba="1 1 0 1"/>
+    </material>
+    <material name="purple">
+        <color rgba="0.5 0 0.5 1"/>
     </material>
     <material name="dark_green">

File: src/my_robot_description/urdf/my_robot_leg.xacro (robot description, xacro)
@@ -84,5 +84,5 @@
         <parent link="servo1"/>
         <child  link="servo1_padding"/>
-        <origin xyz="0 ${-servo_z/2 - 0.002} 0.01125" rpy="0 0 0"/>
+        <origin xyz="0 ${-servo_z/2-0.002} 0.01125" rpy="0 0 0"/>
         <axis xyz="0 1 0"/>
         <limit effort="1000.0" velocity="1.0" lower="${3*urdf_pi/4}" upper="${5*urdf_pi/4}"/>
@@ -151,5 +151,5 @@
         <parent link="servo2"/>
         <child  link="servo2_padding"/>
-        <origin xyz="${servo_z/2 + 0.002} -0.03525 0" rpy="0 0 0"/>
+        <origin xyz="${servo_z/2+0.002} -0.03525 0" rpy="0 0 0"/>
         <axis xyz="1 0 0"/>
         <limit effort="1000.0" velocity="1.0" lower="${3*urdf_pi/4}" upper="${5*urdf_pi/4}"/>
@@ -218,5 +218,50 @@
         <parent link="outer_thigh"/>
         <child  link="servo3"/>
-        <origin xyz="0.010 -0.006 0" rpy="0 0 0"/>
+        <origin xyz="${servo_y/2-0.006-0.0025} -0.004 0" rpy="0 0 0"/>
+    </joint>
+    <link name="calfJoint">
+        <visual>
+            <geometry>
+                <mesh filename="package://my_robot_description/mesh/CADv0/_mod_calfJoint-Body.stl" scale="0.001 0.001 0.001"/>
+            </geometry>
+            <origin xyz="0 0 0" rpy="${-urdf_pi/2} 0 ${urdf_pi/2}"/>
+            <material name="white"/>
+        </visual>
+        <collision>
+            <geometry>
+                <cylinder radius="0.011" length="0.006"/>
+            </geometry>
+            <origin xyz="0 0 0" rpy="0 0 0"/>
+        </collision>
+        <xacro:cylinder_inertia m="0.001" r="0.011" l="0.006" o_xyz="0 0 0" o_rpy="0 0 0"/>
+    </link>
+    <joint name="servo3_calfJoint" type="revolute">
+        <parent link="servo3"/>
+        <child  link="calfJoint"/>
+        <origin xyz="${-servo_z/2-0.0025-0.002} ${-0.011-0.010-0.0025/2} 0" rpy="0 0 0"/>
+        <axis xyz="1 0 0"/>
+        <limit effort="1000.0" velocity="1.0" lower="0" upper="${2*urdf_pi}"/>
+        <dynamics friction="0.05" damping="0.1"/>
+    </joint>
+    <link name="calfFeet">
+        <visual>
+            <geometry>
+                <mesh filename="package://my_robot_description/mesh/CADv0/calfFeet-Body.stl" scale="0.001 0.001 0.001"/>
+            </geometry>
+            <material name="purple"/>
+            <origin xyz="0 0 0" rpy="0 ${-urdf_pi/2} ${urdf_pi}"/>
+        </visual>
+        <collision>
+            <geometry>
+                <box size="0.110 0.040 0.006"/>
+            </geometry>
+            <origin xyz="0.003 -0.055 0" rpy="0 0 0"/>
+        </collision>
+        <xacro:box_inertia m="0.01" x="0.040" y="0.032" z="0.006" o_xyz="0 0 0" o_rpy="0 0 0"/>
+    </link>
+    <joint name="calfJoint_calfFeet" type="fixed">
+        <parent link="calfJoint"/>
+        <child  link="calfFeet"/>
+        <origin xyz="-0.0025 ${-0.09+0.011+0.010+0.0025/2} -0.032" rpy="0 0 0"/>
     </joint>
 </robot>

Commit message: - initial completion of my_robot_leg.xacro, including all the collision geometry and moment of inertia checks

File: src/my_robot_description/urdf/common_properties.xacro (robot description, xacro)
@@ -28,4 +28,7 @@
     <material name="purple">
         <color rgba="0.5 0 0.5 1"/>
+    </material>
+    <material name="dark_purple">
+        <color rgba="0.2 0 0.2 1"/>
     </material>
     <material name="dark_green">

File: src/my_robot_description/urdf/my_robot_leg.xacro (robot description, xacro)
@@ -84,5 +84,5 @@
         <parent link="servo1"/>
         <child  link="servo1_padding"/>
-        <origin xyz="0 ${-servo_z/2-0.002} 0.01125" rpy="0 0 0"/>
+        <origin xyz="0 ${-servo_z/2-0.002} ${0.01+0.0025/2}" rpy="0 0 0"/>
         <axis xyz="0 1 0"/>
         <limit effort="1000.0" velocity="1.0" lower="${3*urdf_pi/4}" upper="${5*urdf_pi/4}"/>
@@ -230,16 +230,16 @@
         <collision>
             <geometry>
-                <cylinder radius="0.011" length="0.006"/>
-            </geometry>
-            <origin xyz="0 0 0" rpy="${-urdf_pi/2} 0 ${urdf_pi/2}"/>
-        </collision>
-        <xacro:cylinder_inertia m="0.001" r="0.011" l="0.006" o_xyz="0 0 0" o_rpy="${-urdf_pi/2} 0 ${urdf_pi/2}"/>
+                <box size="0.022 0.051 0.0065"/>
+            </geometry>
+            <origin xyz="-0.0005 0 -0.0145" rpy="${-urdf_pi/2} 0 ${urdf_pi/2}"/>
+        </collision>
+        <xacro:box_inertia m="0.0015" x="0.022" y="0.051" z="0.0065" o_xyz="-0.0005 0 -0.0145" o_rpy="${-urdf_pi/2} 0 ${urdf_pi/2}"/>
     </link>
     <joint name="servo3_calfJoint" type="revolute">
         <parent link="servo3"/>
         <child  link="calfJoint"/>
-        <origin xyz="${-servo_z/2-0.0025-0.002} ${-0.011-0.010-0.0025/2} 0" rpy="0 0 0"/>
+        <origin xyz="${-servo_z/2-0.002-0.0025} ${-0.01-0.0025/2} 0" rpy="0 0 0"/>
         <axis xyz="1 0 0"/>
-        <limit effort="1000.0" velocity="1.0" lower="${3*urdf_pi/4}" upper="${5*urdf_pi/4}"/>
+        <limit effort="1000.0" velocity="1.0" lower="${5*urdf_pi/8}" upper="${11*urdf_pi/8}"/>
         <dynamics friction="0.05" damping="0.1"/>
     </joint>
@@ -250,22 +250,43 @@
             </geometry>
             <material name="purple"/>
-            <origin xyz="0 0 0" rpy="0 ${-urdf_pi/2} ${urdf_pi}"/>
-        </visual>
-        <collision>
-            <geometry>
-                <box size="0.110 0.040 0.006"/>
-            </geometry>
-            <origin xyz="0.003 -0.055 0" rpy="0 0 0"/>
-        </collision>
-        <xacro:box_inertia m="0.02" x="0.040" y="0.032" z="0.006" o_xyz="0 0 0" o_rpy="0 0 0"/>
+            <origin xyz="0 -0.008 -0.035" rpy="0 ${-urdf_pi/2} 0"/>
+        </visual>
+        <collision>
+            <geometry>
+                <box size="0.150 0.016 0.004"/>
+            </geometry>
+            <origin xyz="-0.002 ${-0.008+0.008} ${-0.035+0.080}" rpy="0 ${-urdf_pi/2} 0"/>
+        </collision>
+        <xacro:box_inertia m="0.02" x="0.150" y="0.016" z="0.004" o_xyz="${-servo_z/2-0.002-0.0025-0.002} ${-0.008+0.008} ${-0.035+0.080}" o_rpy="0 ${-urdf_pi/2} 0"/>
     </link>
     <joint name="servo3_calfFeet" type="revolute">
         <parent link="servo3"/>
         <child  link="calfFeet"/>
-        <origin xyz="-0.0025 ${-0.09+0.011+0.010+0.0025/2} -0.032" rpy="0 0 0"/>
+        <origin xyz="${-servo_z/2-0.002-0.0025} -0.101 0" rpy="0 0 0"/>
         <axis xyz="1 0 0"/>
         <mimic joint="servo3_calfJoint" multiplier="1.0" offset="0.0"/>
-        <limit effort="1000.0" velocity="1.0" lower="${3*urdf_pi/4}" upper="${5*urdf_pi/4}"/>
-        <dynamics friction="0.05" damping="0.1"/>
+        <limit effort="1000.0" velocity="1.0" lower="${5*urdf_pi/8}" upper="${11*urdf_pi/8}"/>
+        <dynamics friction="0.05" damping="0.1"/>
+    </joint>
+    <link name="calfSphere">
+        <visual>
+            <geometry>
+                <sphere radius="0.013"/>
+            </geometry>
+            <origin xyz="0 0 0" rpy="0 0 0"/>
+            <material name="dark_purple"/>
+        </visual>
+        <collision>
+            <geometry>
+                <sphere radius="0.011"/>
+            </geometry>
+            <origin xyz="0 0 0" rpy="0 0 0"/>
+        </collision>
+        <xacro:sphere_inertia m="0.001" r="0.011" o_xyz="0 0 0" o_rpy="0 0 0"/>
+    </link>
+    <joint name="calfFeet_calfSphere" type="fixed">
+        <parent link="calfFeet"/>
+        <child  link="calfSphere"/>
+        <origin xyz="-0.002 0.004 ${0.150-0.035}" rpy="0 0 0"/>
     </joint>
 </robot>
