Commit message: - dimension tunning for base plates and 1 leg

File: src/my_robot_description/urdf/common_properties.xacro (robot description, xacro)
@@ -1,5 +1,5 @@
 <?xml version="1.0"?>
 <robot xmlns:xacro="http://www.ros.org/wiki/xacro">
-    <xacro:property name="urdf_pi" value="3.14159"/>
+    <xacro:property name="urdf_pi" value="3.1415926"/>
     <material name="white">
         <color rgba="1 1 1 1"/>

File: src/my_robot_description/urdf/cubic_doggo.urdf.xacro (robot description, xacro)
@@ -8,25 +8,5 @@
         <visual>
             <geometry>
-                <box size="0.052 0.096 0.06"/>
-            </geometry>
-            <origin xyz="0 0 -0.03" rpy="0 0 0"/>
-            <material name="grey"/>
-        </visual>
-        <collision>
-            <geometry>
-                <box size="0.052 0.096 0.06"/>
-            </geometry>
-            <origin xyz="0 0 -0.03" rpy="0 0 0"/>
-        </collision>
-        <xacro:lazy_inertia m="0.01"/>
-    </link>
-    <joint name="world_base_link" type="fixed">
-        <parent link="world"/>
-        <child link="base_link"/>
-    </joint>
-    <link name="torso">
-        <visual>
-            <geometry>
-                <mesh filename="package://my_robot_description/mesh/CADv0/basePlateTorsoUpper-Body.stl" scale="0.001 0.001 0.001"/>
+                <mesh filename="package://my_robot_description/mesh/CADv0.1/basePlateTorsoUpper-Body.stl" scale="0.001 0.001 0.001"/>
             </geometry>
             <origin xyz="0 0 0" rpy="0 0 0"/>
@@ -35,13 +15,13 @@
         <collision>
             <geometry>
-                <box size="0.132 0.036 0.004"/>
+                <box size="0.056 0.252 0.004"/>
             </geometry>
-            <origin xyz="0 0.018 0.002" rpy="0 0 0"/>
+            <origin xyz="0.0 0.0 0.002" rpy="0 0 0"/>
         </collision>
         <xacro:lazy_inertia m="0.0336"/>
     </link>
-    <joint name="base_link_torso" type="fixed">
-        <parent link="base_link"/>
-        <child  link="torso"/>
+    <joint name="world_base_link" type="fixed">
+        <parent link="world"/>
+        <child  link="base_link"/>
         <origin xyz="0 0 0" rpy="0 0 0"/>
     </joint>
@@ -49,5 +29,5 @@
         <visual>
             <geometry>
-                <mesh filename="package://my_robot_description/mesh/CADv0/basePlate.stl" scale="0.001 0.001 0.001"/>
+                <mesh filename="package://my_robot_description/mesh/CADv0.1/basePlate-Body.stl" scale="0.001 0.001 0.001"/>
             </geometry>
             <origin xyz="0 0 0" rpy="0 0 0"/>
@@ -56,5 +36,5 @@
         <collision>
             <geometry>
-                <box size="0.132 0.036 0.004"/>
+                <box size="0.141 0.036 0.004"/>
             </geometry>
             <origin xyz="0 0.018 0.002" rpy="0 0 0"/>
@@ -63,12 +43,12 @@
     </link>
     <joint name="torso_base_plate_F" type="fixed">
-        <parent link="torso"/>
+        <parent link="base_link"/>
         <child  link="base_plate_F"/>
-        <origin xyz="0 0.012 -0.004" rpy="0 0 0"/>
+        <origin xyz="0 0.09 0.004" rpy="0 0 0"/>
     </joint>
     <link name="base_plate_B">
         <visual>
             <geometry>
-                <mesh filename="package://my_robot_description/mesh/CADv0/basePlate.stl" scale="0.001 0.001 0.001"/>
+                <mesh filename="package://my_robot_description/mesh/CADv0.1/basePlate-Body.stl" scale="0.001 0.001 0.001"/>
             </geometry>
             <origin xyz="0 0 0" rpy="0 0 0"/>
@@ -77,5 +57,5 @@
         <collision>
             <geometry>
-                <box size="0.132 0.036 0.004"/>
+                <box size="0.141 0.036 0.004"/>
             </geometry>
             <origin xyz="0 0.018 0.002" rpy="0 0 0"/>
@@ -84,13 +64,13 @@
     </link>
     <joint name="torso_base_plate_B" type="fixed">
-        <parent link="torso"/>
+        <parent link="base_link"/>
         <child  link="base_plate_B"/>
-        <origin xyz="0 -0.012 -0.004" rpy="0 0 0"/>
+        <origin xyz="0 -0.066 0.004" rpy="0 0 0"/>
     </joint>
 <!-- ================================================================================================================================== -->
     <xacro:doggo_leg prefix='FR'/>
-    <xacro:doggo_leg prefix='FL'/>
+    <!--xacro:doggo_leg prefix='FL'/>
     <xacro:doggo_leg prefix='BR'/>
-    <xacro:doggo_leg prefix='BL'/>
+    <xacro:doggo_leg prefix='BL'/-->
 <!-- ================================================================================================================================== -->
 </robot>

File: src/my_robot_description/urdf/cubic_doggo_leg.xacro (robot description, xacro)
@@ -9,5 +9,5 @@
         <xacro:property name="rflc"              value=" 1"/>
         <xacro:property name="base_plate"        value="base_plate_F"/>
-        <xacro:property name="servo1_holder_xyz" value=" 0.026  0.048 0"/>
+        <xacro:property name="servo1_holder_xyz" value="-0.052 0.018 0.004"/>
     </xacro:if>
     <xacro:if value="${prefix == 'FL'}">
@@ -37,5 +37,5 @@
         <collision>
             <geometry>
-                <box size="0.037 0.032 0.014"/>
+                <box size="0.037 0.037 0.014"/>
             </geometry>
             <origin xyz="0 0 0.007" rpy="0 0 ${rflc*urdf_pi/2}"/>
@@ -104,5 +104,5 @@
         <collision>
             <geometry>
-                <box size="0.037 0.032 0.014"/>
+                <box size="0.037 0.037 0.014"/>
             </geometry>
             <origin xyz="0 -0.007 0" rpy="${rflc*urdf_pi/2} 0 0"/>
@@ -193,5 +193,5 @@
         <collision>
             <geometry>
-                <box size="0.110 0.040 0.006"/>
+                <box size="0.080 0.040 0.006"/>
             </geometry>
             <origin xyz="${rflc*0.003} -0.055 0" rpy="${-rflc*urdf_pi/2} 0 ${-rflc*urdf_pi/2}"/>
@@ -233,11 +233,11 @@
             </geometry>
             <material name="purple"/>
-            <origin xyz="${-rflc*0.004} -0.008 0.035" rpy="0 ${urdf_pi/2} 0"/>
-        </visual>
-        <collision>
-            <geometry>
-                <box size="0.150 0.016 0.004"/>
-            </geometry>
-            <origin xyz="${-rflc*0.002} ${-0.008+0.008} ${0.035-0.080}" rpy="0 ${-urdf_pi/2} 0"/>
+            <origin xyz="${-rflc*0.004} -0.008 0.038" rpy="0 ${urdf_pi/2} 0"/>
+        </visual>
+        <collision>
+            <geometry>
+                <box size="0.110 0.016 0.004"/>
+            </geometry>
+            <origin xyz="0 ${-0.008+0.008} ${0.038-0.050}" rpy="0 ${-urdf_pi/2} 0"/>
         </collision>
         <xacro:box_inertia m="${0.0251-0.0080}" x="0.150" y="0.016" z="0.004"
@@ -247,5 +247,5 @@
         <parent link="servo3_${prefix}"/>
         <child  link="calfFeet_${prefix}"/>
-        <origin xyz="${rflc*(-servo_z/2-0.002-0.0025)} ${-0.101+0.004} 0" rpy="0 0 0"/>
+        <origin xyz="${rflc*(-servo_z/2-0.002-0.0025)} ${-0.086+0.004} 0" rpy="0 0 0"/>
         <axis xyz="${-rflc} 0 0"/>
         <limit effort="1000.0" velocity="20.0" lower="2.0" upper="4.0"/>
@@ -262,7 +262,7 @@
         <collision>
             <geometry>
-                <box size="0.022 0.051 0.0065"/>
-            </geometry>
-            <origin xyz="${-rflc*0.0005} 0 0.0145" rpy="${rflc*urdf_pi/2} 0 ${-rflc*urdf_pi/2}"/>
+                <box size="0.022 0.053 0.007"/>
+            </geometry>
+            <origin xyz="${-rflc*0.0005} 0 0.0155" rpy="${rflc*urdf_pi/2} 0 ${-rflc*urdf_pi/2}"/>
         </collision>
         <xacro:box_inertia m="${0.0047+0.0015}" x="0.022" y="0.051" z="0.0065"
@@ -297,5 +297,5 @@
         <parent link="calfFeet_${prefix}"/>
         <child  link="calfSphere_${prefix}"/>
-        <origin xyz="${-rflc*0.002} 0.004 ${-0.150+0.035}" rpy="0 0 0"/>
+        <origin xyz="0 0.004 ${-0.105+0.035}" rpy="0 0 0"/>
     </joint>
     </xacro:macro>
