Commit message: - debugged moveit demo for cubic_doggo

File: src/my_robot_description/urdf/cubic_doggo.ros2_control.xacro (robot description, xacro)
@@ -1,132 +1,164 @@
 <?xml version="1.0"?>
 <robot xmlns:xacro="http://www.ros.org/wiki/xacro">
-    <xacro:macro name="cubic_doggo_ros2_control" params="name initial_positions_file">
-        <xacro:property name="initial_positions" value="${xacro.load_yaml(initial_positions_file)['initial_positions']}"/>
-        <ros2_control name="${name}" type="system">
-            <hardware>
-                <!-- By default, set up controllers for simulation. This won't work on real hardware -->
-                <plugin>mock_components/GenericSystem</plugin>
-            </hardware>
-            <joint name="servo1_servo1_padding_FR">
-                <command_interface name="position"/>
-                <command_interface name="velocity"/>
-                <command_interface name="effort"/>
-                <state_interface name="position">
-                  <param name="initial_value">${initial_positions['servo1_servo1_padding_FR']}</param>
-                </state_interface>
-                <state_interface name="velocity"/>
-                <state_interface name="effort"/>
-            </joint>
-            <joint name="servo2_servo2_padding_FR">
-                <command_interface name="position"/>
-                <command_interface name="velocity"/>
-                <command_interface name="effort"/>
-                <state_interface name="position">
-                  <param name="initial_value">${initial_positions['servo2_servo2_padding_FR']}</param>
-                </state_interface>
-                <state_interface name="velocity"/>
-                <state_interface name="effort"/>
-            </joint>
-            <joint name="servo3_calfFeet_FR">
-                <command_interface name="position"/>
-                <command_interface name="velocity"/>
-                <command_interface name="effort"/>
-                <state_interface name="position">
-                  <param name="initial_value">${initial_positions['servo3_calfFeet_FR']}</param>
-                </state_interface>
-                <state_interface name="velocity"/>
-                <state_interface name="effort"/>
-            </joint>
-            <joint name="servo1_servo1_padding_FL">
-                <command_interface name="position"/>
-                <command_interface name="velocity"/>
-                <command_interface name="effort"/>
-                <state_interface name="position">
-                  <param name="initial_value">${initial_positions['servo1_servo1_padding_FL']}</param>
-                </state_interface>
-                <state_interface name="velocity"/>
-                <state_interface name="effort"/>
-            </joint>
-            <joint name="servo2_servo2_padding_FL">
-                <command_interface name="position"/>
-                <command_interface name="velocity"/>
-                <command_interface name="effort"/>
-                <state_interface name="position">
-                  <param name="initial_value">${initial_positions['servo2_servo2_padding_FL']}</param>
-                </state_interface>
-                <state_interface name="velocity"/>
-                <state_interface name="effort"/>
-            </joint>
-            <joint name="servo3_calfFeet_FL">
-                <command_interface name="position"/>
-                <command_interface name="velocity"/>
-                <command_interface name="effort"/>
-                <state_interface name="position">
-                  <param name="initial_value">${initial_positions['servo3_calfFeet_FL']}</param>
-                </state_interface>
-                <state_interface name="velocity"/>
-                <state_interface name="effort"/>
-            </joint>
-            <joint name="servo1_servo1_padding_BR">
-                <command_interface name="position"/>
-                <command_interface name="velocity"/>
-                <command_interface name="effort"/>
-                <state_interface name="position">
-                  <param name="initial_value">${initial_positions['servo1_servo1_padding_BR']}</param>
-                </state_interface>
-                <state_interface name="velocity"/>
-                <state_interface name="effort"/>
-            </joint>
-            <joint name="servo2_servo2_padding_BR">
-                <command_interface name="position"/>
-                <command_interface name="velocity"/>
-                <command_interface name="effort"/>
-                <state_interface name="position">
-                  <param name="initial_value">${initial_positions['servo2_servo2_padding_BR']}</param>
-                </state_interface>
-                <state_interface name="velocity"/>
-                <state_interface name="effort"/>
-            </joint>
-            <joint name="servo3_calfFeet_BR">
-                <command_interface name="position"/>
-                <command_interface name="velocity"/>
-                <command_interface name="effort"/>
-                <state_interface name="position">
-                  <param name="initial_value">${initial_positions['servo3_calfFeet_BR']}</param>
-                </state_interface>
-                <state_interface name="velocity"/>
-                <state_interface name="effort"/>
-            </joint>
-            <joint name="servo1_servo1_padding_BL">
-                <command_interface name="position"/>
-                <command_interface name="velocity"/>
-                <command_interface name="effort"/>
-                <state_interface name="position">
-                  <param name="initial_value">${initial_positions['servo1_servo1_padding_BL']}</param>
-                </state_interface>
-                <state_interface name="velocity"/>
-                <state_interface name="effort"/>
-            </joint>
-            <joint name="servo2_servo2_padding_BL">
-                <command_interface name="position"/>
-                <command_interface name="velocity"/>
-                <command_interface name="effort"/>
-                <state_interface name="position">
-                  <param name="initial_value">${initial_positions['servo2_servo2_padding_BL']}</param>
-                </state_interface>
-                <state_interface name="velocity"/>
-                <state_interface name="effort"/>
-            </joint>
-            <joint name="servo3_calfFeet_BL">
-                <command_interface name="position"/>
-                <command_interface name="velocity"/>
-                <command_interface name="effort"/>
-                <state_interface name="position">
-                  <param name="initial_value">${initial_positions['servo3_calfFeet_BL']}</param>
-                </state_interface>
-                <state_interface name="velocity"/>
-                <state_interface name="effort"/>
-            </joint>
-        </ros2_control>
-    </xacro:macro>
+    <ros2_control name="cubic_doggo_controller" type="system">
+        <hardware>
+            <plugin>mock_components/GenericSystem</plugin>
+            <param name="servo1_channel_FR">11</param>
+            <param name="servo2_channel_FR">12</param>
+            <param name="servo3_channel_FR">13</param>
+            <param name="servo1_channel_FL">11</param>
+            <param name="servo2_channel_FL">12</param>
+            <param name="servo3_channel_FL">13</param>
+            <param name="servo1_channel_GR">11</param>
+            <param name="servo2_channel_GR">12</param>
+            <param name="servo3_channel_GR">13</param>
+            <param name="servo1_channel_GL">11</param>
+            <param name="servo2_channel_GL">12</param>
+            <param name="servo3_channel_GL">13</param>
+        </hardware>
+        <joint name="servo1_servo1_padding_FR">
+            <command_interface name="position"/>
+            <state_interface name="position">
+              <param name="initial_value">3.14</param>
+            </state_interface>
+            <state_interface name="velocity">
+              <param name="initial_value">0.0</param>
+            </state_interface>
+            <state_interface name="effort">
+              <param name="initial_value">0.0</param>
+            </state_interface>
+        </joint>
+        <joint name="servo2_servo2_padding_FR">
+            <command_interface name="position"/>
+            <state_interface name="position">
+              <param name="initial_value">3.14</param>
+            </state_interface>
+            <state_interface name="velocity">
+              <param name="initial_value">0.0</param>
+            </state_interface>
+            <state_interface name="effort">
+              <param name="initial_value">0.0</param>
+            </state_interface>
+        </joint>
+        <joint name="servo3_calfFeet_FR">
+            <command_interface name="position"/>
+            <state_interface name="position">
+              <param name="initial_value">3.14</param>
+            </state_interface>
+            <state_interface name="velocity">
+              <param name="initial_value">0.0</param>
+            </state_interface>
+            <state_interface name="effort">
+              <param name="initial_value">0.0</param>
+            </state_interface>
+        </joint>
+        <joint name="servo1_servo1_padding_FL">
+            <command_interface name="position"/>
+            <state_interface name="position">
+              <param name="initial_value">3.14</param>
+            </state_interface>
+            <state_interface name="velocity">
+              <param name="initial_value">0.0</param>
+            </state_interface>
+            <state_interface name="effort">
+              <param name="initial_value">0.0</param>
+            </state_interface>
+        </joint>
+        <joint name="servo2_servo2_padding_FL">
+            <command_interface name="position"/>
+            <state_interface name="position">
+              <param name="initial_value">3.14</param>
+            </state_interface>
+            <state_interface name="velocity">
+              <param name="initial_value">0.0</param>
+            </state_interface>
+            <state_interface name="effort">
+              <param name="initial_value">0.0</param>
+            </state_interface>
+        </joint>
+        <joint name="servo3_calfFeet_FL">
+            <command_interface name="position"/>
+            <state_interface name="position">
+              <param name="initial_value">3.14</param>
+            </state_interface>
+            <state_interface name="velocity">
+              <param name="initial_value">0.0</param>
+            </state_interface>
+            <state_interface name="effort">
+              <param name="initial_value">0.0</param>
+            </state_interface>
+        </joint>
+        <joint name="servo1_servo1_padding_BR">
+            <command_interface name="position"/>
+            <state_interface name="position">
+              <param name="initial_value">3.14</param>
+            </state_interface>
+            <state_interface name="velocity">
+              <param name="initial_value">0.0</param>
+            </state_interface>
+            <state_interface name="effort">
+              <param name="initial_value">0.0</param>
+            </state_interface>
+        </joint>
+        <joint name="servo2_servo2_padding_BR">
+            <command_interface name="position"/>
+            <state_interface name="position">
+              <param name="initial_value">3.14</param>
+            </state_interface>
+            <state_interface name="velocity">
+              <param name="initial_value">0.0</param>
+            </state_interface>
+            <state_interface name="effort">
+              <param name="initial_value">0.0</param>
+            </state_interface>
+        </joint>
+        <joint name="servo3_calfFeet_BR">
+            <command_interface name="position"/>
+            <state_interface name="position">
+              <param name="initial_value">3.14</param>
+            </state_interface>
+            <state_interface name="velocity">
+              <param name="initial_value">0.0</param>
+            </state_interface>
+            <state_interface name="effort">
+              <param name="initial_value">0.0</param>
+            </state_interface>
+        </joint>
+        <joint name="servo1_servo1_padding_BL">
+            <command_interface name="position"/>
+            <state_interface name="position">
+              <param name="initial_value">3.14</param>
+            </state_interface>
+            <state_interface name="velocity">
+              <param name="initial_value">0.0</param>
+            </state_interface>
+            <state_interface name="effort">
+              <param name="initial_value">0.0</param>
+            </state_interface>
+        </joint>
+        <joint name="servo2_servo2_padding_BL">
+            <command_interface name="position"/>
+            <state_interface name="position">
+              <param name="initial_value">3.14</param>
+            </state_interface>
+            <state_interface name="velocity">
+              <param name="initial_value">0.0</param>
+            </state_interface>
+            <state_interface name="effort">
+              <param name="initial_value">0.0</param>
+            </state_interface>
+        </joint>
+        <joint name="servo3_calfFeet_BL">
+            <command_interface name="position"/>
+            <state_interface name="position">
+              <param name="initial_value">3.14</param>
+            </state_interface>
+            <state_interface name="velocity">
+              <param name="initial_value">0.0</param>
+            </state_interface>
+            <state_interface name="effort">
+              <param name="initial_value">0.0</param>
+            </state_interface>
+        </joint>
+    </ros2_control>
 </robot>

File: src/my_robot_description/urdf/cubic_doggo.urdf.xacro (robot description, xacro)
@@ -3,4 +3,5 @@
     <xacro:include filename="common_properties.xacro"/>
     <xacro:include filename="cubic_doggo_leg.xacro"/>
+    <xacro:include filename="cubic_doggo.ros2_control.xacro"/>
 <!-- ================================================================================================================================== -->
     <link name="world"/>

Commit message: - correct some label mismatches

File: src/my_robot_description/urdf/cubic_doggo.ros2_control.xacro (robot description, xacro)
@@ -5,17 +5,53 @@
             <!--plugin>mock_components/GenericSystem</plugin-->
             <plugin>cubic_doggo_namespace/HardwareInterfaceU2D2_cubic_doggo</plugin>
-            <param name="servo1_channel_FR">11</param>
-            <param name="servo2_channel_FR">12</param>
-            <param name="servo3_channel_FR">13</param>
-            <param name="servo1_channel_FL">21</param>
-            <param name="servo2_channel_FL">22</param>
-            <param name="servo3_channel_FL">23</param>
-            <param name="servo1_channel_BR">31</param>
-            <param name="servo2_channel_BR">32</param>
-            <param name="servo3_channel_BR">33</param>
-            <param name="servo1_channel_BL">41</param>
-            <param name="servo2_channel_BL">42</param>
-            <param name="servo3_channel_BL">43</param>
+            <param name="servo1_channel_FL">11</param>
+            <param name="servo2_channel_FL">12</param>
+            <param name="servo3_channel_FL">13</param>
+            <param name="servo1_channel_FR">21</param>
+            <param name="servo2_channel_FR">22</param>
+            <param name="servo3_channel_FR">23</param>
+            <param name="servo1_channel_BL">31</param>
+            <param name="servo2_channel_BL">32</param>
+            <param name="servo3_channel_BL">33</param>
+            <param name="servo1_channel_BR">41</param>
+            <param name="servo2_channel_BR">42</param>
+            <param name="servo3_channel_BR">43</param>
         </hardware>
+        <joint name="servo1_servo1_padding_FL">
+            <command_interface name="position"/>
+            <state_interface name="position">
+              <param name="initial_value">3.14</param>
+            </state_interface>
+            <state_interface name="velocity">
+              <param name="initial_value">0.0</param>
+            </state_interface>
+            <state_interface name="effort">
+              <param name="initial_value">0.0</param>
+            </state_interface>
+        </joint>
+        <joint name="servo2_servo2_padding_FL">
+            <command_interface name="position"/>
+            <state_interface name="position">
+              <param name="initial_value">3.14</param>
+            </state_interface>
+            <state_interface name="velocity">
+              <param name="initial_value">0.0</param>
+            </state_interface>
+            <state_interface name="effort">
+              <param name="initial_value">0.0</param>
+            </state_interface>
+        </joint>
+        <joint name="servo3_calfFeet_FL">
+            <command_interface name="position"/>
+            <state_interface name="position">
+              <param name="initial_value">3.14</param>
+            </state_interface>
+            <state_interface name="velocity">
+              <param name="initial_value">0.0</param>
+            </state_interface>
+            <state_interface name="effort">
+              <param name="initial_value">0.0</param>
+            </state_interface>
+        </joint>
         <joint name="servo1_servo1_padding_FR">
             <command_interface name="position"/>
@@ -54,5 +90,5 @@
             </state_interface>
         </joint>
-        <joint name="servo1_servo1_padding_FL">
+        <joint name="servo1_servo1_padding_BL">
             <command_interface name="position"/>
             <state_interface name="position">
@@ -66,5 +102,5 @@
             </state_interface>
         </joint>
-        <joint name="servo2_servo2_padding_FL">
+        <joint name="servo2_servo2_padding_BL">
             <command_interface name="position"/>
             <state_interface name="position">
@@ -78,5 +114,5 @@
             </state_interface>
         </joint>
-        <joint name="servo3_calfFeet_FL">
+        <joint name="servo3_calfFeet_BL">
             <command_interface name="position"/>
             <state_interface name="position">
@@ -126,40 +162,4 @@
             </state_interface>
         </joint>
-        <joint name="servo1_servo1_padding_BL">
-            <command_interface name="position"/>
-            <state_interface name="position">
-              <param name="initial_value">3.14</param>
-            </state_interface>
-            <state_interface name="velocity">
-              <param name="initial_value">0.0</param>
-            </state_interface>
-            <state_interface name="effort">
-              <param name="initial_value">0.0</param>
-            </state_interface>
-        </joint>
-        <joint name="servo2_servo2_padding_BL">
-            <command_interface name="position"/>
-            <state_interface name="position">
-              <param name="initial_value">3.14</param>
-            </state_interface>
-            <state_interface name="velocity">
-              <param name="initial_value">0.0</param>
-            </state_interface>
-            <state_interface name="effort">
-              <param name="initial_value">0.0</param>
-            </state_interface>
-        </joint>
-        <joint name="servo3_calfFeet_BL">
-            <command_interface name="position"/>
-            <state_interface name="position">
-              <param name="initial_value">3.14</param>
-            </state_interface>
-            <state_interface name="velocity">
-              <param name="initial_value">0.0</param>
-            </state_interface>
-            <state_interface name="effort">
-              <param name="initial_value">0.0</param>
-            </state_interface>
-        </joint>
     </ros2_control>
 </robot>
