Commit message: - successfully running 4 legs in urdf

File: src/my_robot_description/urdf/cubic_doggo.urdf.xacro (robot description, xacro)
@@ -26,8 +26,8 @@
     </joint>
 <!-- ================================================================================================================================== -->
-    <xacro:doggo_leg prefix="FR" origin_xyz="0.026 0.048 0"/>
-    <xacro:doggo_leg prefix="FL" origin_xyz="0.026 -0.048 0"/>
-    <xacro:doggo_leg prefix="RR" origin_xyz="-0.026 0.048 0"/>
-    <xacro:doggo_leg prefix="RL" origin_xyz="-0.026 -0.048 0"/>
+    <xacro:doggo_leg prefix='FR'/>
+    <xacro:doggo_leg prefix='FL'/>
+    <xacro:doggo_leg prefix='BR'/>
+    <xacro:doggo_leg prefix='BL'/>
 <!-- ================================================================================================================================== -->
 </robot>

File: src/my_robot_description/urdf/cubic_doggo_leg.xacro (robot description, xacro)
@@ -289,4 +289,5 @@
         <origin xyz="-0.002 0.004 ${-0.150+0.035}" rpy="0 0 0"/>
     </joint>
+    </xacro:macro>
 </robot>
 <!-- ================================================================================================================================== -->

Commit message: - overall geometry adjustment for base plates

File: src/my_robot_description/urdf/cubic_doggo.urdf.xacro (robot description, xacro)
@@ -25,4 +25,67 @@
         <child link="base_link"/>
     </joint>
+    <link name="torso">
+        <visual>
+            <geometry>
+                <mesh filename="package://my_robot_description/mesh/CADv0/basePlateTorsoUpper-Body.stl" scale="0.001 0.001 0.001"/>
+            </geometry>
+            <origin xyz="0 0 0" rpy="0 0 0"/>
+            <material name="grey"/>
+        </visual>
+        <collision>
+            <geometry>
+                <box size="0.132 0.036 0.004"/>
+            </geometry>
+            <origin xyz="0 0.018 0.002" rpy="0 0 0"/>
+        </collision>
+        <xacro:lazy_inertia m="0.0336"/>
+    </link>
+    <joint name="base_link_torso" type="fixed">
+        <parent link="base_link"/>
+        <child  link="torso"/>
+        <origin xyz="0 0 0" rpy="0 0 0"/>
+    </joint>
+    <link name="base_plate_F">
+        <visual>
+            <geometry>
+                <mesh filename="package://my_robot_description/mesh/CADv0/basePlate.stl" scale="0.001 0.001 0.001"/>
+            </geometry>
+            <origin xyz="0 0 0" rpy="0 0 0"/>
+            <material name="grey"/>
+        </visual>
+        <collision>
+            <geometry>
+                <box size="0.132 0.036 0.004"/>
+            </geometry>
+            <origin xyz="0 0.018 0.002" rpy="0 0 0"/>
+        </collision>
+        <xacro:lazy_inertia m="0.0336"/>
+    </link>
+    <joint name="torso_base_plate_F" type="fixed">
+        <parent link="torso"/>
+        <child  link="base_plate_F"/>
+        <origin xyz="0 0.012 -0.004" rpy="0 0 0"/>
+    </joint>
+    <link name="base_plate_B">
+        <visual>
+            <geometry>
+                <mesh filename="package://my_robot_description/mesh/CADv0/basePlate.stl" scale="0.001 0.001 0.001"/>
+            </geometry>
+            <origin xyz="0 0 0" rpy="0 0 0"/>
+            <material name="grey"/>
+        </visual>
+        <collision>
+            <geometry>
+                <box size="0.132 0.036 0.004"/>
+            </geometry>
+            <origin xyz="0 0.018 0.002" rpy="0 0 0"/>
+        </collision>
+        <xacro:lazy_inertia m="0.0336"/>
+    </link>
+    <joint name="torso_base_plate_B" type="fixed">
+        <parent link="torso"/>
+        <child  link="base_plate_B"/>
+        <origin xyz="0 -0.012 -0.004" rpy="0 0 0"/>
+    </joint>
 <!-- ================================================================================================================================== -->
     <xacro:doggo_leg prefix="FR" origin_xyz="0.026 0.048 0"/>

File: src/my_robot_description/urdf/cubic_doggo_leg.xacro (robot description, xacro)
@@ -7,13 +7,21 @@
     <xacro:property name="servo_z" value="0.034"/>
     <xacro:if value="${prefix == 'FR'}">
+        <xacro:property name="rflc"              value=" 1"/>
+        <xacro:property name="base_plate"        value="base_plate_F"/>
         <xacro:property name="servo1_holder_xyz" value=" 0.026  0.048 0"/>
     </xacro:if>
     <xacro:if value="${prefix == 'FL'}">
+        <xacro:property name="rflc"              value="-1"/>
+        <xacro:property name="base_plate"        value="base_plate_F"/>
         <xacro:property name="servo1_holder_xyz" value="-0.026  0.048 0"/>
     </xacro:if>
     <xacro:if value="${prefix == 'BR'}">
+        <xacro:property name="rflc"              value=" 1"/>
+        <xacro:property name="base_plate"        value='base_plate_B'/>
         <xacro:property name="servo1_holder_xyz" value=" 0.026 -0.048 0"/>
     </xacro:if>
     <xacro:if value="${prefix == 'BL'}">
+        <xacro:property name="rflc"              value="-1"/>
+        <xacro:property name="base_plate"        value='base_plate_B'/>
         <xacro:property name="servo1_holder_xyz" value="-0.026 -0.048 0"/>
     </xacro:if>
@@ -25,5 +33,5 @@
             </geometry>
             <material name="white"/>
-            <origin xyz="0 0 0" rpy="0 0 ${urdf_pi/2}"/>
+            <origin xyz="0 0 0" rpy="0 0 ${rflc*urdf_pi/2}"/>
         </visual>
         <collision>
@@ -31,10 +39,10 @@
                 <box size="0.037 0.032 0.014"/>
             </geometry>
-            <origin xyz="0 0 0.007" rpy="0 0 ${urdf_pi/2}"/>
-        </collision>
-        <xacro:box_inertia m="0.0098" x="0.037" y="0.032" z="0.014" o_xyz="0 0 0.007" o_rpy="0 0 ${urdf_pi/2}"/>
-    </link>
-    <joint name="main_board_servo1_holder_${prefix}" type="fixed">
-        <parent link="base_link"/>
+            <origin xyz="0 0 0.007" rpy="0 0 ${rflc*urdf_pi/2}"/>
+        </collision>
+        <xacro:box_inertia m="0.0098" x="0.037" y="0.032" z="0.014" o_xyz="0 0 0.007" o_rpy="0 0 ${rflc*urdf_pi/2}"/>
+    </link>
+    <joint name="base_plate_servo1_holder_${prefix}" type="fixed">
+        <parent link="${base_plate}"/>
         <child  link="servo1_holder_${prefix}"/>
         <origin xyz="${servo1_holder_xyz}" rpy="0 0 0"/>
@@ -112,5 +120,5 @@
                 <box size="${servo_x} ${servo_y} ${servo_z}"/>
             </geometry>
-            <origin xyz="0 ${-servo_y/2} 0" rpy="0 ${urdf_pi/2} 0"/>
+            <origin xyz="0 ${-servo_y/2} 0" rpy="0 ${rflc*urdf_pi/2} 0"/>
             <material name="black"/>
         </visual>
@@ -119,7 +127,8 @@
                 <box size="${servo_x} ${servo_y} ${servo_z}"/>
             </geometry>
-            <origin xyz="0 ${-servo_y/2} 0" rpy="0 ${urdf_pi/2} 0"/>
-        </collision>
-        <xacro:box_inertia m="0.0572" x="${servo_x}" y="${servo_y}" z="${servo_z}" o_xyz="0 ${-servo_y/2} 0" o_rpy="0 ${urdf_pi/2} 0"/>
+            <origin xyz="0 ${-servo_y/2} 0" rpy="0 ${rflc*urdf_pi/2} 0"/>
+        </collision>
+        <xacro:box_inertia m="0.0572" x="${servo_x}" y="${servo_y}" z="${servo_z}"
+                           o_xyz="0 ${-servo_y/2} 0" o_rpy="0 ${rflc*urdf_pi/2} 0"/>
     </link>
     <joint name="servo2_holder_servo2_${prefix}" type="fixed">
@@ -133,5 +142,5 @@
                 <cylinder radius="0.011" length="0.004"/>
             </geometry>
-            <origin xyz="0.002 0 0" rpy="0 ${urdf_pi/2} 0"/>
+            <origin xyz="${rflc*0.002} 0 0" rpy="0 ${rflc*urdf_pi/2} 0"/>
             <material name="white"/>
         </visual>
@@ -140,12 +149,12 @@
                 <cylinder radius="0.011" length="0.004"/>
             </geometry>
-            <origin xyz="0.002 0 0" rpy="0 ${urdf_pi/2} 0"/>
-        </collision>
-        <xacro:cylinder_inertia m="0.0013" r="0.011" l="0.004" o_xyz="0.002 0 0" o_rpy="0 ${urdf_pi/2} 0"/>
+            <origin xyz="${rflc*0.002} 0 0" rpy="0 ${rflc*urdf_pi/2} 0"/>
+        </collision>
+        <xacro:cylinder_inertia m="0.0013" r="0.011" l="0.004" o_xyz="${rflc*0.002} 0 0" o_rpy="0 ${rflc*urdf_pi/2} 0"/>
     </link>
     <joint name="servo2_servo2_padding_${prefix}" type="revolute">
         <parent link="servo2_${prefix}"/>
         <child  link="servo2_padding_${prefix}"/>
-        <origin xyz="${servo_z/2+0.002} -0.03525 0" rpy="0 0 0"/>
+        <origin xyz="${rflc*(servo_z/2+0.002)} -0.03525 0" rpy="0 0 0"/>
         <axis xyz="1 0 0"/>
         <limit effort="1000.0" velocity="20.0" lower="2.0" upper="4.0"/>
@@ -159,5 +168,5 @@
             </geometry>
             <material name="blue"/>
-            <origin xyz="0 0 0" rpy="${-urdf_pi/2} 0 ${-urdf_pi/2}"/>
+            <origin xyz="0 0 0" rpy="${-urdf_pi/2} 0 ${-rflc*urdf_pi/2}"/>
         </visual>
         <collision>
@@ -165,12 +174,13 @@
                 <box size="0.032 0.040 0.006"/>
             </geometry>
-            <origin xyz="0.003 -0.016 0" rpy="${-urdf_pi/2} 0 ${-urdf_pi/2}"/>
-        </collision>
-        <xacro:box_inertia m="0.0085" x="0.040" y="0.032" z="0.006" o_xyz="0.003 -0.016 0" o_rpy="${-urdf_pi/2} 0 ${-urdf_pi/2}"/>
+            <origin xyz="${rflc*0.003} -0.016 0" rpy="${-urdf_pi/2} 0 ${-rflc*urdf_pi/2}"/>
+        </collision>
+        <xacro:box_inertia m="0.0085" x="0.040" y="0.032" z="0.006"
+                           o_xyz="${rflc*0.003} -0.016 0" o_rpy="${-urdf_pi/2} 0 ${-rflc*urdf_pi/2}"/>
     </link>
     <joint name="servo2_padding_inner_thigh_${prefix}" type="fixed">
         <parent link="servo2_padding_${prefix}"/>
         <child  link="inner_thigh_${prefix}"/>
-        <origin xyz="0.004 0.016 0" rpy="0 0 0"/>
+        <origin xyz="${rflc*0.004} 0.016 0" rpy="0 0 0"/>
     </joint>
     <link name="outer_thigh_${prefix}">
@@ -180,5 +190,5 @@
             </geometry>
             <material name="blue"/>
-            <origin xyz="0 0 0" rpy="${-urdf_pi/2} 0 ${-urdf_pi/2}"/>
+            <origin xyz="0 0 0" rpy="${-urdf_pi/2} 0 ${-rflc*urdf_pi/2}"/>
         </visual>
         <collision>
@@ -186,12 +196,13 @@
                 <box size="0.110 0.040 0.006"/>
             </geometry>
-            <origin xyz="0.003 -0.055 0" rpy="${-urdf_pi/2} 0 ${-urdf_pi/2}"/>
-        </collision>
-        <xacro:box_inertia m="0.0113" x="0.040" y="0.032" z="0.006" o_xyz="0.003 -0.055 0" o_rpy="${-urdf_pi/2} 0 ${-urdf_pi/2}"/>
+            <origin xyz="${rflc*0.003} -0.055 0" rpy="${-urdf_pi/2} 0 ${-rflc*urdf_pi/2}"/>
+        </collision>
+        <xacro:box_inertia m="0.0113" x="0.040" y="0.032" z="0.006"
+                           o_xyz="${rflc*0.003} -0.055 0" o_rpy="${-urdf_pi/2} 0 ${-rflc*urdf_pi/2}"/>
     </link>
     <joint name="inner_thigh_outer_thigh_${prefix}" type="fixed">
         <parent link="inner_thigh_${prefix}"/>
         <child  link="outer_thigh_${prefix}"/>
-        <origin xyz="0.028 0 0" rpy="0 0 0"/>
+        <origin xyz="${rflc*0.028} 0 0" rpy="0 0 0"/>
     </joint>
     <link name="servo3_${prefix}">
@@ -200,5 +211,5 @@
                 <box size="${servo_x} ${servo_y} ${servo_z}"/>
             </geometry>
-            <origin xyz="0 ${-servo_y/2} 0" rpy="0 ${urdf_pi/2} 0"/>
+            <origin xyz="0 ${-servo_y/2} 0" rpy="0 ${rflc*urdf_pi/2} 0"/>
             <material name="black"/>
         </visual>
@@ -207,13 +218,13 @@
                 <box size="${servo_x} ${servo_y} ${servo_z}"/>
             </geometry>
-            <origin xyz="0 ${-servo_y/2} 0" rpy="0 ${urdf_pi/2} 0"/>
+            <origin xyz="0 ${-servo_y/2} 0" rpy="0 ${rflc*urdf_pi/2} 0"/>
         </collision>
         <xacro:box_inertia m="${0.0572+0.0113+0.0078}" x="${servo_x}" y="${servo_y}" z="${servo_z}"
-                           o_xyz="0 ${-servo_y/2} 0" o_rpy="0 ${urdf_pi/2} 0"/>
+                           o_xyz="0 ${-servo_y/2} 0" o_rpy="0 ${rflc*urdf_pi/2} 0"/>
     </link>
     <joint name="outer_thigh_servo3_${prefix}" type="fixed">
         <parent link="outer_thigh_${prefix}"/>
         <child  link="servo3_${prefix}"/>
-        <origin xyz="${servo_y/2-0.006-0.0025} -0.004 0" rpy="0 0 0"/>
+        <origin xyz="${rflc*(servo_y/2-0.006-0.0025)} -0.004 0" rpy="0 0 0"/>
     </joint>
     <link name="calfFeet_${prefix}">
@@ -223,5 +234,5 @@
             </geometry>
             <material name="purple"/>
-            <origin xyz="-0.004 -0.008 0.035" rpy="0 ${urdf_pi/2} 0"/>
+            <origin xyz="${-rflc*0.004} -0.008 0.035" rpy="0 ${rflc*urdf_pi/2} 0"/>
         </visual>
         <collision>
@@ -229,13 +240,13 @@
                 <box size="0.150 0.016 0.004"/>
             </geometry>
-            <origin xyz="-0.002 ${-0.008+0.008} ${0.035-0.080}" rpy="0 ${-urdf_pi/2} 0"/>
+            <origin xyz="${-rflc*0.002} ${-0.008+0.008} ${0.035-0.080}" rpy="0 ${-rflc*urdf_pi/2} 0"/>
         </collision>
         <xacro:box_inertia m="${0.0251-0.0080}" x="0.150" y="0.016" z="0.004"
-                           o_xyz="${-servo_z/2-0.002-0.0025-0.002} ${-0.008+0.008} ${0.035-0.080}" o_rpy="0 ${-urdf_pi/2} 0"/>
+                           o_xyz="${rflc*(-servo_z/2-0.002-0.0025-0.002)} ${-0.008+0.008} ${0.035-0.080}" o_rpy="0 ${-rflc*urdf_pi/2} 0"/>
     </link>
     <joint name="servo3_calfFeet_${prefix}" type="revolute">
         <parent link="servo3_${prefix}"/>
         <child  link="calfFeet_${prefix}"/>
-        <origin xyz="${-servo_z/2-0.002-0.0025} ${-0.101+0.004} 0" rpy="0 0 0"/>
+        <origin xyz="${rflc*(-servo_z/2-0.002-0.0025)} ${-0.101+0.004} 0" rpy="0 0 0"/>
         <axis xyz="-1 0 0"/>
         <limit effort="1000.0" velocity="20.0" lower="2.0" upper="4.0"/>
@@ -247,5 +258,5 @@
                 <mesh filename="package://my_robot_description/mesh/CADv0.1/calfJoint-Body.stl" scale="0.001 0.001 0.001"/>
             </geometry>
-            <origin xyz="0 0 0" rpy="${urdf_pi/2} 0 ${-urdf_pi/2}"/>
+            <origin xyz="0 0 0" rpy="${urdf_pi/2} 0 ${-rflc*urdf_pi/2}"/>
             <material name="white"/>
         </visual>
@@ -254,13 +265,13 @@
                 <box size="0.022 0.051 0.0065"/>
             </geometry>
-            <origin xyz="-0.0005 0 0.0145" rpy="${urdf_pi/2} 0 ${-urdf_pi/2}"/>
+            <origin xyz="${-rflc*0.0005} 0 0.0145" rpy="${urdf_pi/2} 0 ${-rflc*urdf_pi/2}"/>
         </collision>
         <xacro:box_inertia m="${0.0047+0.0015}" x="0.022" y="0.051" z="0.0065"
-                           o_xyz="-0.0005 0 0.0145" o_rpy="${urdf_pi/2} 0 ${-urdf_pi/2}"/>
+                           o_xyz="${-rflc*0.0005} 0 0.0145" o_rpy="${urdf_pi/2} 0 ${-rflc*urdf_pi/2}"/>
     </link>
     <joint name="servo3_calfJoint_${prefix}" type="revolute">
         <parent link="servo3_${prefix}"/>
         <child  link="calfJoint_${prefix}"/>
-        <origin xyz="${-servo_z/2-0.002-0.0025} ${-0.01-0.0025/2} 0" rpy="0 0 0"/>
+        <origin xyz="${rflc*(-servo_z/2-0.002-0.0025)} ${-0.01-0.0025/2} 0" rpy="0 0 0"/>
         <axis xyz="-1 0 0"/>
         <mimic joint="servo3_calfFeet_${prefix}" multiplier="1.0" offset="0.0"/>
@@ -287,5 +298,5 @@
         <parent link="calfFeet_${prefix}"/>
         <child  link="calfSphere_${prefix}"/>
-        <origin xyz="-0.002 0.004 ${-0.150+0.035}" rpy="0 0 0"/>
+        <origin xyz="${-rflc*0.002} 0.004 ${-0.150+0.035}" rpy="0 0 0"/>
     </joint>
 </robot>
