Commit message: - update the dimension/revolution for reflected leg

File: src/my_robot_description/urdf/cubic_doggo.urdf.xacro (robot description, xacro)
@@ -70,6 +70,6 @@
 <!-- ================================================================================================================================== -->
     <xacro:doggo_leg prefix='FR'/>
-    <!--xacro:doggo_leg prefix='FL'/>
-    <xacro:doggo_leg prefix='BR'/>
+    <xacro:doggo_leg prefix='FL'/>
+    <!--xacro:doggo_leg prefix='BR'/>
     <xacro:doggo_leg prefix='BL'/-->
 <!-- ================================================================================================================================== -->

File: src/my_robot_description/urdf/cubic_doggo_leg.xacro (robot description, xacro)
@@ -14,5 +14,5 @@
         <xacro:property name="rflc"              value="-1"/>
         <xacro:property name="base_plate"        value="base_plate_F"/>
-        <xacro:property name="servo1_holder_xyz" value="-0.026  0.048 0"/>
+        <xacro:property name="servo1_holder_xyz" value=" 0.052 0.018 0.004"/>
     </xacro:if>
     <xacro:if value="${prefix == 'BR'}">
@@ -33,5 +33,5 @@
             </geometry>
             <material name="white"/>
-            <origin xyz="0 0 0" rpy="0 0 ${rflc*urdf_pi/2}"/>
+            <origin xyz="0 0 0" rpy="0 0 ${urdf_pi/2}"/>
         </visual>
         <collision>
@@ -39,7 +39,7 @@
                 <box size="0.037 0.037 0.014"/>
             </geometry>
-            <origin xyz="0 0 0.007" rpy="0 0 ${rflc*urdf_pi/2}"/>
-        </collision>
-        <xacro:box_inertia m="0.0098" x="0.037" y="0.032" z="0.014" o_xyz="0 0 0.007" o_rpy="0 0 ${rflc*urdf_pi/2}"/>
+            <origin xyz="0 0 0.007" rpy="0 0 ${urdf_pi/2}"/>
+        </collision>
+        <xacro:box_inertia m="0.0098" x="0.037" y="0.032" z="0.014" o_xyz="0 0 0.007" o_rpy="0 0 ${urdf_pi/2}"/>
     </link>
     <joint name="base_plate_servo1_holder_${prefix}" type="fixed">
@@ -53,5 +53,5 @@
                 <box size="${servo_x} ${servo_y} ${servo_z}"/>
             </geometry>
-            <origin xyz="0 0 ${servo_y/2}" rpy="${rflc*urdf_pi/2} 0 0"/>
+            <origin xyz="0 0 ${servo_y/2}" rpy="${urdf_pi/2} 0 0"/>
             <material name="black"/>
         </visual>
@@ -60,7 +60,7 @@
                 <box size="${servo_x} ${servo_y} ${servo_z}"/>
             </geometry>
-            <origin xyz="0 0 ${servo_y/2}" rpy="${rflc*urdf_pi/2} 0 0"/>
-        </collision>
-        <xacro:box_inertia m="0.0572" x="${servo_x}" y="${servo_y}" z="${servo_z}" o_xyz="0 0 ${servo_y/2}" o_rpy="${rflc*urdf_pi/2} 0 0"/>
+            <origin xyz="0 0 ${servo_y/2}" rpy="${urdf_pi/2} 0 0"/>
+        </collision>
+        <xacro:box_inertia m="0.0572" x="${servo_x}" y="${servo_y}" z="${servo_z}" o_xyz="0 0 ${servo_y/2}" o_rpy="${urdf_pi/2} 0 0"/>
     </link>
     <joint name="servo1_holder_servo1_${prefix}" type="fixed">
@@ -74,5 +74,5 @@
                 <cylinder radius="0.011" length="0.004"/>
             </geometry>
-            <origin xyz="0 -0.002 0" rpy="${rflc*urdf_pi/2} 0 0"/>
+            <origin xyz="0 -0.002 0" rpy="${urdf_pi/2} 0 0"/>
             <material name="white"/>
         </visual>
@@ -81,7 +81,7 @@
                 <cylinder radius="0.011" length="0.004"/>
             </geometry>
-            <origin xyz="0 -0.002 0" rpy="${rflc*urdf_pi/2} 0 0"/>
-        </collision>
-        <xacro:cylinder_inertia m="0.0013" r="0.011" l="0.004" o_xyz="0 -0.002 0" o_rpy="${rflc*urdf_pi/2} 0 0"/>
+            <origin xyz="0 -0.002 0" rpy="${urdf_pi/2} 0 0"/>
+        </collision>
+        <xacro:cylinder_inertia m="0.0013" r="0.011" l="0.004" o_xyz="0 -0.002 0" o_rpy="${urdf_pi/2} 0 0"/>
     </link>
     <joint name="servo1_servo1_padding_${prefix}" type="revolute">
@@ -90,5 +90,5 @@
         <origin xyz="0 ${-servo_z/2-0.002} ${0.01+0.0025/2}" rpy="0 0 0"/>
         <axis xyz="0 -1 0"/>
-        <limit effort="1000.0" velocity="20.0" lower="2.5" upper="4.0"/>
+        <limit effort="1000.0" velocity="20.0" lower="${urdf_pi - urdf_pi/3}" upper="${urdf_pi + urdf_pi/3}"/>
         <dynamics friction="0.05" damping="0.1"/>
     </joint>
@@ -100,5 +100,5 @@
             </geometry>
             <material name="white"/>
-            <origin xyz="0 0 0" rpy="${rflc*urdf_pi/2} 0 0"/>
+            <origin xyz="0 0 0" rpy="${urdf_pi/2} 0 0"/>
         </visual>
         <collision>
@@ -106,7 +106,7 @@
                 <box size="0.037 0.037 0.014"/>
             </geometry>
-            <origin xyz="0 -0.007 0" rpy="${rflc*urdf_pi/2} 0 0"/>
-        </collision>
-        <xacro:box_inertia m="0.0098" x="0.037" y="0.032" z="0.014" o_xyz="0 -0.007 0" o_rpy="${rflc*urdf_pi/2} 0 0"/>
+            <origin xyz="0 -0.007 0" rpy="${urdf_pi/2} 0 0"/>
+        </collision>
+        <xacro:box_inertia m="0.0098" x="0.037" y="0.032" z="0.014" o_xyz="0 -0.007 0" o_rpy="${urdf_pi/2} 0 0"/>
     </link>
     <joint name="base_link_servo2_holder_${prefix}" type="fixed">
@@ -120,5 +120,5 @@
                 <box size="${servo_x} ${servo_y} ${servo_z}"/>
             </geometry>
-            <origin xyz="0 ${-servo_y/2} 0" rpy="0 ${urdf_pi/2} 0"/>
+            <origin xyz="0 ${-servo_y/2} 0" rpy="0 ${rflc*urdf_pi/2} 0"/>
             <material name="black"/>
         </visual>
@@ -127,7 +127,7 @@
                 <box size="${servo_x} ${servo_y} ${servo_z}"/>
             </geometry>
-            <origin xyz="0 ${-servo_y/2} 0" rpy="0 ${urdf_pi/2} 0"/>
-        </collision>
-        <xacro:box_inertia m="0.0572" x="${servo_x}" y="${servo_y}" z="${servo_z}" o_xyz="0 ${-servo_y/2} 0" o_rpy="0 ${urdf_pi/2} 0"/>
+            <origin xyz="0 ${-servo_y/2} 0" rpy="0 ${rflc*urdf_pi/2} 0"/>
+        </collision>
+        <xacro:box_inertia m="0.0572" x="${servo_x}" y="${servo_y}" z="${servo_z}" o_xyz="0 ${-servo_y/2} 0" o_rpy="0 ${rflc*urdf_pi/2} 0"/>
     </link>
     <joint name="servo2_holder_servo2_${prefix}" type="fixed">
@@ -157,5 +157,6 @@
         <origin xyz="${rflc*(servo_z/2+0.002)} -0.03525 0" rpy="0 0 0"/>
         <axis xyz="${rflc} 0 0"/>
-        <limit effort="1000.0" velocity="20.0" lower="2.0" upper="4.0"/>
+        <limit effort="1000.0" velocity="20.0" lower="${urdf_pi - 2*urdf_pi/6 - rflc*urdf_pi/6}"
+                                               upper="${urdf_pi + 2*urdf_pi/6 - rflc*urdf_pi/6}"/>
         <dynamics friction="0.05" damping="0.1"/>
     </joint>
@@ -167,5 +168,5 @@
             </geometry>
             <material name="blue"/>
-            <origin xyz="0 0 0" rpy="${-rflc*urdf_pi/2} 0 ${-rflc*urdf_pi/2}"/>
+            <origin xyz="0 0 0" rpy="${-rflc*urdf_pi/2} 0 ${-urdf_pi/2}"/>
         </visual>
         <collision>
@@ -173,8 +174,8 @@
                 <box size="0.032 0.040 0.006"/>
             </geometry>
-            <origin xyz="${rflc*0.003} -0.016 0" rpy="${-rflc*urdf_pi/2} 0 ${-rflc*urdf_pi/2}"/>
+            <origin xyz="${rflc*0.003} -0.016 0" rpy="${-rflc*urdf_pi/2} 0 ${-urdf_pi/2}"/>
         </collision>
         <xacro:box_inertia m="0.0085" x="0.040" y="0.032" z="0.006"
-                           o_xyz="${rflc*0.003} -0.016 0" o_rpy="${-rflc*urdf_pi/2} 0 ${-rflc*urdf_pi/2}"/>
+                           o_xyz="${rflc*0.003} -0.016 0" o_rpy="${-rflc*urdf_pi/2} 0 ${-urdf_pi/2}"/>
     </link>
     <joint name="servo2_padding_inner_thigh_${prefix}" type="fixed">
@@ -189,14 +190,14 @@
             </geometry>
             <material name="blue"/>
-            <origin xyz="0 0 0" rpy="${-rflc*urdf_pi/2} 0 ${-rflc*urdf_pi/2}"/>
-        </visual>
-        <collision>
-            <geometry>
-                <box size="0.080 0.040 0.006"/>
-            </geometry>
-            <origin xyz="${rflc*0.003} -0.055 0" rpy="${-rflc*urdf_pi/2} 0 ${-rflc*urdf_pi/2}"/>
+            <origin xyz="0 0 0" rpy="${-urdf_pi/2} ${urdf_pi/2-rflc*urdf_pi/2} ${-rflc*urdf_pi/2}"/>
+        </visual>
+        <collision>
+            <geometry>
+                <box size="0.095 0.040 0.006"/>
+            </geometry>
+            <origin xyz="${rflc*0.003} -0.0475 0" rpy="${-urdf_pi/2} ${urdf_pi/2-rflc*urdf_pi/2} ${-rflc*urdf_pi/2}"/>
         </collision>
         <xacro:box_inertia m="0.0113" x="0.040" y="0.032" z="0.006"
-                           o_xyz="${rflc*0.003} -0.055 0" o_rpy="${-rflc*urdf_pi/2} 0 ${-rflc*urdf_pi/2}"/>
+                           o_xyz="${rflc*0.003} -0.055 0" o_rpy="${-urdf_pi/2} ${urdf_pi/2-rflc*urdf_pi/2} ${-rflc*urdf_pi/2}"/>
     </link>
     <joint name="inner_thigh_outer_thigh_${prefix}" type="fixed">
@@ -210,5 +211,5 @@
                 <box size="${servo_x} ${servo_y} ${servo_z}"/>
             </geometry>
-            <origin xyz="0 ${-servo_y/2} 0" rpy="0 ${urdf_pi/2} 0"/>
+            <origin xyz="0 ${-servo_y/2} 0" rpy="0 ${rflc*urdf_pi/2} 0"/>
             <material name="black"/>
         </visual>
@@ -217,8 +218,8 @@
                 <box size="${servo_x} ${servo_y} ${servo_z}"/>
             </geometry>
-            <origin xyz="0 ${-servo_y/2} 0" rpy="0 ${urdf_pi/2} 0"/>
+            <origin xyz="0 ${-servo_y/2} 0" rpy="0 ${rflc*urdf_pi/2} 0"/>
         </collision>
         <xacro:box_inertia m="${0.0572+0.0113+0.0078}" x="${servo_x}" y="${servo_y}" z="${servo_z}"
-                           o_xyz="0 ${-servo_y/2} 0" o_rpy="0 ${urdf_pi/2} 0"/>
+                           o_xyz="0 ${-servo_y/2} 0" o_rpy="0 ${rflc*urdf_pi/2} 0"/>
     </link>
     <joint name="outer_thigh_servo3_${prefix}" type="fixed">
@@ -233,5 +234,5 @@
             </geometry>
             <material name="purple"/>
-            <origin xyz="${-rflc*0.004} -0.008 0.038" rpy="0 ${urdf_pi/2} 0"/>
+            <origin xyz="${-0.004} -0.008 0.038" rpy="0 ${urdf_pi/2} 0"/>
         </visual>
         <collision>
@@ -249,5 +250,5 @@
         <origin xyz="${rflc*(-servo_z/2-0.002-0.0025)} ${-0.086+0.004} 0" rpy="0 0 0"/>
         <axis xyz="${-rflc} 0 0"/>
-        <limit effort="1000.0" velocity="20.0" lower="2.0" upper="4.0"/>
+        <limit effort="1000.0" velocity="20.0" lower="${5*urdf_pi/8}" upper="${11*urdf_pi/8}"/>
         <dynamics friction="0.05" damping="0.1"/>
     </joint>
@@ -257,5 +258,5 @@
                 <mesh filename="package://my_robot_description/mesh/CADv0.1/calfJoint-Body.stl" scale="0.001 0.001 0.001"/>
             </geometry>
-            <origin xyz="0 0 0" rpy="${rflc*urdf_pi/2} 0 ${-rflc*urdf_pi/2}"/>
+            <origin xyz="0 0 0" rpy="${urdf_pi/2} 0 ${-rflc*urdf_pi/2}"/>
             <material name="white"/>
         </visual>
@@ -264,8 +265,8 @@
                 <box size="0.022 0.053 0.007"/>
             </geometry>
-            <origin xyz="${-rflc*0.0005} 0 0.0155" rpy="${rflc*urdf_pi/2} 0 ${-rflc*urdf_pi/2}"/>
+            <origin xyz="${-rflc*0.0005} 0 0.0155" rpy="${urdf_pi/2} 0 ${-rflc*urdf_pi/2}"/>
         </collision>
         <xacro:box_inertia m="${0.0047+0.0015}" x="0.022" y="0.051" z="0.0065"
-                           o_xyz="${-rflc*0.0005} 0 0.0145" o_rpy="${rflc*urdf_pi/2} 0 ${-rflc*urdf_pi/2}"/>
+                           o_xyz="${-rflc*0.0005} 0 0.0145" o_rpy="${urdf_pi/2} 0 ${-rflc*urdf_pi/2}"/>
     </link>
     <joint name="servo3_calfJoint_${prefix}" type="revolute">

Commit message: - adding all 4 legs in urdf

File: src/my_robot_description/urdf/cubic_doggo.urdf.xacro (robot description, xacro)
@@ -69,8 +69,8 @@
     </joint>
 <!-- ================================================================================================================================== -->
+    <xacro:doggo_leg prefix='FL'/>
     <xacro:doggo_leg prefix='FR'/>
-    <xacro:doggo_leg prefix='FL'/>
-    <!--xacro:doggo_leg prefix='BR'/>
-    <xacro:doggo_leg prefix='BL'/-->
+    <xacro:doggo_leg prefix='BL'/>
+    <xacro:doggo_leg prefix='BR'/>
 <!-- ================================================================================================================================== -->
 </robot>

File: src/my_robot_description/urdf/cubic_doggo_leg.xacro (robot description, xacro)
@@ -6,23 +6,23 @@
     <xacro:property name="servo_y" value="0.0465"/>
     <xacro:property name="servo_z" value="0.034"/>
-    <xacro:if value="${prefix == 'FR'}">
+    <xacro:if value="${prefix == 'FL'}">
         <xacro:property name="rflc"              value=" 1"/>
         <xacro:property name="base_plate"        value="base_plate_F"/>
         <xacro:property name="servo1_holder_xyz" value="-0.052 0.018 0.004"/>
     </xacro:if>
-    <xacro:if value="${prefix == 'FL'}">
+    <xacro:if value="${prefix == 'FR'}">
         <xacro:property name="rflc"              value="-1"/>
         <xacro:property name="base_plate"        value="base_plate_F"/>
         <xacro:property name="servo1_holder_xyz" value=" 0.052 0.018 0.004"/>
     </xacro:if>
-    <xacro:if value="${prefix == 'BR'}">
+    <xacro:if value="${prefix == 'BL'}">
         <xacro:property name="rflc"              value=" 1"/>
         <xacro:property name="base_plate"        value='base_plate_B'/>
-        <xacro:property name="servo1_holder_xyz" value=" 0.026 -0.048 0"/>
+        <xacro:property name="servo1_holder_xyz" value="-0.052 0.018 0"/>
     </xacro:if>
-    <xacro:if value="${prefix == 'BL'}">
+    <xacro:if value="${prefix == 'BR'}">
         <xacro:property name="rflc"              value="-1"/>
         <xacro:property name="base_plate"        value='base_plate_B'/>
-        <xacro:property name="servo1_holder_xyz" value="-0.026 -0.048 0"/>
+        <xacro:property name="servo1_holder_xyz" value=" 0.052 0.018 0"/>
     </xacro:if>
     <!-- ============================================================================================================================== -->

Commit message: - initial moveit configs for cubic_doggo

File: src/my_robot_description/urdf/cubic_doggo.urdf.xacro (robot description, xacro)
@@ -1,4 +1,4 @@
 <?xml version="1.0"?>
-<robot name="cubic_doggoV0" xmlns:xacro="http://www.ros.org/wiki/xacro">
+<robot name="cubic_doggo" xmlns:xacro="http://www.ros.org/wiki/xacro">
     <xacro:include filename="common_properties.xacro"/>
     <xacro:include filename="cubic_doggo_leg.xacro"/>
@@ -45,5 +45,5 @@
         <parent link="base_link"/>
         <child  link="base_plate_F"/>
-        <origin xyz="0 0.09 0.004" rpy="0 0 0"/>
+        <origin xyz="0 -0.066 0.004" rpy="0 0 0"/>
     </joint>
     <link name="base_plate_B">
@@ -66,5 +66,5 @@
         <parent link="base_link"/>
         <child  link="base_plate_B"/>
-        <origin xyz="0 -0.066 0.004" rpy="0 0 0"/>
+        <origin xyz="0 0.09 0.004" rpy="0 0 0"/>
     </joint>
 <!-- ================================================================================================================================== -->

File: src/my_robot_description/urdf/cubic_doggo_leg.xacro (robot description, xacro)
@@ -19,10 +19,10 @@
         <xacro:property name="rflc"              value=" 1"/>
         <xacro:property name="base_plate"        value='base_plate_B'/>
-        <xacro:property name="servo1_holder_xyz" value="-0.052 0.018 0"/>
+        <xacro:property name="servo1_holder_xyz" value="-0.052 0.018 0.004"/>
     </xacro:if>
     <xacro:if value="${prefix == 'BR'}">
         <xacro:property name="rflc"              value="-1"/>
         <xacro:property name="base_plate"        value='base_plate_B'/>
-        <xacro:property name="servo1_holder_xyz" value=" 0.052 0.018 0"/>
+        <xacro:property name="servo1_holder_xyz" value=" 0.052 0.018 0.004"/>
     </xacro:if>
     <!-- ============================================================================================================================== -->

Commit message: - changes require to be loaded into Isaac Sim

File: src/my_robot_description/urdf/cubic_doggo.urdf.xacro (robot description, xacro)
@@ -9,5 +9,5 @@
         <visual>
             <geometry>
-                <mesh filename="package://my_robot_description/mesh/CADv0.1/basePlateTorsoUpper-Body.stl" scale="0.001 0.001 0.001"/>
+                <mesh filename="package://my_robot_description/mesh/CADv0.1/basePlateTorsoUpper.stl" scale="0.001 0.001 0.001"/>
             </geometry>
             <origin xyz="0 0 0" rpy="0 0 0"/>
@@ -30,5 +30,5 @@
         <visual>
             <geometry>
-                <mesh filename="package://my_robot_description/mesh/CADv0.1/basePlate-Body.stl" scale="0.001 0.001 0.001"/>
+                <mesh filename="package://my_robot_description/mesh/CADv0.1/basePlate.stl" scale="0.001 0.001 0.001"/>
             </geometry>
             <origin xyz="0 0 0" rpy="0 0 0"/>
@@ -51,5 +51,5 @@
         <visual>
             <geometry>
-                <mesh filename="package://my_robot_description/mesh/CADv0.1/basePlate-Body.stl" scale="0.001 0.001 0.001"/>
+                <mesh filename="package://my_robot_description/mesh/CADv0.1/basePlate.stl" scale="0.001 0.001 0.001"/>
             </geometry>
             <origin xyz="0 0 0" rpy="0 0 0"/>

File: src/my_robot_description/urdf/cubic_doggo_leg.xacro (robot description, xacro)
@@ -30,5 +30,5 @@
         <visual>
             <geometry>
-                <mesh filename="package://my_robot_description/mesh/CADv0.1/XL-430holderBasic-Body.stl" scale="0.001 0.001 0.001"/>
+                <mesh filename="package://my_robot_description/mesh/CADv0.1/XL430holderBasic.stl" scale="0.001 0.001 0.001"/>
             </geometry>
             <material name="white"/>
@@ -97,5 +97,5 @@
         <visual>
             <geometry>
-                <mesh filename="package://my_robot_description/mesh/CADv0.1/XL-430holderBasic-Body.stl" scale="0.001 0.001 0.001"/>
+                <mesh filename="package://my_robot_description/mesh/CADv0.1/XL430holderBasic.stl" scale="0.001 0.001 0.001"/>
             </geometry>
             <material name="white"/>
@@ -165,5 +165,5 @@
         <visual>
             <geometry>
-                <mesh filename="package://my_robot_description/mesh/CADv0.1/thighInner-Body.stl" scale="0.001 0.001 0.001"/>
+                <mesh filename="package://my_robot_description/mesh/CADv0.1/thighInner.stl" scale="0.001 0.001 0.001"/>
             </geometry>
             <material name="blue"/>
@@ -187,5 +187,5 @@
         <visual>
             <geometry>
-                <mesh filename="package://my_robot_description/mesh/CADv0.1/thighOuter-Body.stl" scale="0.001 0.001 0.001"/>
+                <mesh filename="package://my_robot_description/mesh/CADv0.1/thighOuter.stl" scale="0.001 0.001 0.001"/>
             </geometry>
             <material name="blue"/>
@@ -256,5 +256,5 @@
         <visual>
             <geometry>
-                <mesh filename="package://my_robot_description/mesh/CADv0.1/calfJoint-Body.stl" scale="0.001 0.001 0.001"/>
+                <mesh filename="package://my_robot_description/mesh/CADv0.1/calfJoint.stl" scale="0.001 0.001 0.001"/>
             </geometry>
             <origin xyz="0 0 0" rpy="${urdf_pi/2} 0 ${-rflc*urdf_pi/2}"/>

Commit message: - now leg_set_name and leg_set_joint work

File: src/my_robot_description/urdf/cubic_doggo.urdf.xacro (robot description, xacro)
@@ -20,5 +20,5 @@
             <origin xyz="0.0 0.0 0.002" rpy="0 0 0"/>
         </collision>
-        <xacro:lazy_inertia m="0.0336"/>
+        <xacro:box_inertia m="0.06" x="0.056" y="0.252" z="0.004" o_xyz="0 0 0.002" o_rpy="0 0 0"/>
     </link>
     <joint name="world_base_link" type="fixed">
@@ -41,5 +41,5 @@
             <origin xyz="0 0.018 0.002" rpy="0 0 0"/>
         </collision>
-        <xacro:lazy_inertia m="0.0336"/>
+        <xacro:box_inertia m="0.0336" x="0.141" y="0.036" z="0.004" o_xyz="0 0.018 0.002" o_rpy="0 0 0"/>
     </link>
     <joint name="torso_base_plate_F" type="fixed">
@@ -62,5 +62,5 @@
             <origin xyz="0 0.018 0.002" rpy="0 0 0"/>
         </collision>
-        <xacro:lazy_inertia m="0.0336"/>
+        <xacro:box_inertia m="0.0336" x="0.141" y="0.036" z="0.004" o_xyz="0 0.018 0.002" o_rpy="0 0 0"/>
     </link>
     <joint name="torso_base_plate_B" type="fixed">

File: src/my_robot_description/urdf/cubic_doggo_leg.xacro (robot description, xacro)
@@ -251,5 +251,5 @@
         <axis xyz="${-rflc} 0 0"/>
         <limit effort="1000.0" velocity="20.0" lower="${5*urdf_pi/8}" upper="${11*urdf_pi/8}"/>
-        <dynamics friction="0.05" damping="0.1"/>
+        <dynamics friction="0.0128" damping="0.1"/>
     </joint>
     <link name="calfJoint_${prefix}">
@@ -277,5 +277,5 @@
         <mimic joint="servo3_calfFeet_${prefix}" multiplier="1.0" offset="0.0"/>
         <limit effort="1000.0" velocity="20.0" lower="${5*urdf_pi/8}" upper="${11*urdf_pi/8}"/>
-        <dynamics friction="0.05" damping="0.1"/>
+        <dynamics friction="0.0212" damping="0.1"/>
     </joint>
     <link name="calfSphere_${prefix}">
